File: kicad/revA/offramps/offramps.kicad_pcb (KiCad board)
At the start: 4 copper layers, 218 x 132 mm, 89 parts, among them J15 Conn_02x06_Odd_Even, J16 Conn_01x24_Female, J17 Conn_01x24_Female, J19 Conn_01x06_Male, J23 Screw_Terminal_01x02, J24 Conn_01x03_Male, J25 Screw_Terminal_01x02, J3 Conn_01x04_Pin, J4 Conn_01x01, U1 MCP4725xxx-xCH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

Commit message: Redactions for paper submission of artifact
Parts:
- J1, J2: footprint jblocklove_kicad:arduino_mega_shield -> jb_kicad:arduino_mega_shield
- J3: footprint jblocklove_kicad:3-way_jumper -> jb_kicad:3-way_jumper
Other:
- board text added: "OffRAMPS"
- board text removed: "JBlocklove"
- board text removed: "NYU PCB - OffRAMPS"
Changed lines of the file:
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@@
     )
   )
-  (footprint "jblocklove_kicad:arduino_mega_shield" (layer "F.Cu")
+  (footprint "jb_kicad:arduino_mega_shield" (layer "F.Cu")
     (at 393.226471 80.842)
     (descr "https://docs.arduino.cc/hardware/mega-2560")
@@
     )
   )
-  (footprint "jblocklove_kicad:3-way_jumper" (layer "F.Cu")
+  (footprint "jb_kicad:3-way_jumper" (layer "F.Cu")
     (at 304.3 180.767447)
     (property "Sheetfile" "cmods7_trojan_shield.kicad_sch")
@@
     )
   )
-  (footprint "jblocklove_kicad:arduino_mega_shield" (layer "F.Cu")
+  (footprint "jb_kicad:arduino_mega_shield" (layer "F.Cu")
     (at 203.996471 80.842)
     (descr "https://docs.arduino.cc/hardware/mega-2560")
@@
   (gr_arc (start 404 68) (mid 406.828427 69.171573) (end 408 72)
     (stroke (width 0.15) (type default)) (layer "Edge.Cuts"))
-  (gr_text "NYU PCB - OffRAMPS" (at 327.8 72) (layer "F.SilkS")
+  (gr_text "OffRAMPS" (at 327.8 72) (layer "F.SilkS")
     (effects (font (size 2.8 2.8) (thickness 0.5) italic))
   )
@@
     (effects (font (size 1.5 1.5) (thickness 0.3)))
   )
-  (gr_text "JBlocklove" (at 367.6 73.9) (layer "F.SilkS")
-    (effects (font (size 2.8 2.8) (thickness 0.5) bold italic) (justify left bottom))
-  )
   (gr_text "Heating FET goes here" (at 351.8 188.4) (layer "F.SilkS")
