File: kicad/revA/offramps/offramps.kicad_sch (KiCad schematic)
At the start: 89 parts, among them J15 Conn_02x06_Odd_Even, J16 Conn_01x24_Female, J17 Conn_01x24_Female, J19 Conn_01x06_Male, J23 Screw_Terminal_01x02, J24 Conn_01x03_Male, J25 Screw_Terminal_01x02, J3 Conn_01x04_Pin, J4 Conn_01x01, U1 MCP4725xxx-xCH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

Commit message: Redactions for paper submission of artifact
Parts:
- J1, J2: footprint jblocklove_kicad:arduino_mega_shield -> jb_kicad:arduino_mega_shield; symbol jblocklove_kicad:atmega_headers -> jb_kicad:atmega_headers
- J3: footprint jblocklove_kicad:3-way_jumper -> jb_kicad:3-way_jumper
Changed lines of the file:
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@@
     )
   )
-  (symbol (lib_name "atmega_headers_3") (lib_id "jblocklove_kicad:atmega_headers") (at 133.35 102.87 0) (unit 4)
+  (symbol (lib_name "atmega_headers_3") (lib_id "jb_kicad:atmega_headers") (at 133.35 102.87 0) (unit 4)
     (in_bom yes) (on_board yes) (dnp no) (fields_autoplaced)
     (property "Reference" "J2" (at 95.25 126.365 0)
@@
       (effects (font (size 1.27 1.27)))
     )
-    (property "Footprint" "jblocklove_kicad:arduino_mega_shield" (at 154.94 125.73 90)
+    (property "Footprint" "jb_kicad:arduino_mega_shield" (at 154.94 125.73 90)
       (effects (font (size 1.27 1.27)) hide)
     )
@@
       (effects (font (size 1.27 1.27)))
     )
-    (property "Footprint" "jblocklove_kicad:3-way_jumper" (at 347.345 50.8 0)
+    (property "Footprint" "jb_kicad:3-way_jumper" (at 347.345 50.8 0)
       (effects (font (size 1.27 1.27)) hide)
     )
@@
     )
   )
-  (symbol (lib_name "atmega_headers_2") (lib_id "jblocklove_kicad:atmega_headers") (at 41.275 27.305 0) (unit 7)
+  (symbol (lib_name "atmega_headers_2") (lib_id "jb_kicad:atmega_headers") (at 41.275 27.305 0) (unit 7)
     (in_bom yes) (on_board yes) (dnp no) (fields_autoplaced)
     (property "Reference" "J1" (at 46.99 42.8982 0)
@@
       (effects (font (size 1.27 1.27)))
     )
-    (property "Footprint" "jblocklove_kicad:arduino_mega_shield" (at 62.865 50.165 90)
+    (property "Footprint" "jb_kicad:arduino_mega_shield" (at 62.865 50.165 90)
       (effects (font (size 1.27 1.27)) hide)
     )
@@
     )
   )
-  (symbol (lib_name "atmega_headers_2") (lib_id "jblocklove_kicad:atmega_headers") (at 42.545 104.775 0) (mirror y) (unit 4)
+  (symbol (lib_name "atmega_headers_2") (lib_id "jb_kicad:atmega_headers") (at 42.545 104.775 0) (mirror y) (unit 4)
     (in_bom yes) (on_board yes) (dnp no) (fields_autoplaced)
     (property "Reference" "J1" (at 27.94 128.27 0)
@@
       (effects (font (size 1.27 1.27)))
     )
-    (property "Footprint" "jblocklove_kicad:arduino_mega_shield" (at 20.955 127.635 90)
+    (property "Footprint" "jb_kicad:arduino_mega_shield" (at 20.955 127.635 90)
       (effects (font (size 1.27 1.27)) hide)
     )
@@
     )
   )
-  (symbol (lib_name "atmega_headers_2") (lib_id "jblocklove_kicad:atmega_headers") (at 59.055 32.385 0) (mirror y) (unit 1)
+  (symbol (lib_name "atmega_headers_2") (lib_id "jb_kicad:atmega_headers") (at 59.055 32.385 0) (mirror y) (unit 1)
     (in_bom yes) (on_board yes) (dnp no) (fields_autoplaced)
     (property "Reference" "J1" (at 59.0549 32.385 0)
@@
       (effects (font (size 1.27 1.27)))
     )
-    (property "Footprint" "jblocklove_kicad:arduino_mega_shield" (at 37.465 55.245 90)
+    (property "Footprint" "jb_kicad:arduino_mega_shield" (at 37.465 55.245 90)
       (effects (font (size 1.27 1.27)) hide)
     )
@@
     )
   )
-  (symbol (lib_name "atmega_headers_2") (lib_id "jblocklove_kicad:atmega_headers") (at 40.005 85.725 0) (unit 5)
+  (symbol (lib_name "atmega_headers_2") (lib_id "jb_kicad:atmega_headers") (at 40.005 85.725 0) (unit 5)
     (in_bom yes) (on_board yes) (dnp no) (fields_autoplaced)
     (property "Reference" "J1" (at 46.99 98.7782 0)
@@
       (effects (font (size 1.27 1.27)))
     )
-    (property "Footprint" "jblocklove_kicad:arduino_mega_shield" (at 61.595 108.585 90)
+    (property "Footprint" "jb_kicad:arduino_mega_shield" (at 61.595 108.585 90)
       (effects (font (size 1.27 1.27)) hide)
     )
@@
     )
   )
-  (symbol (lib_name "atmega_headers_3") (lib_id "jblocklove_kicad:atmega_headers") (at 134.62 82.55 0) (mirror y) (unit 5)
+  (symbol (lib_name "atmega_headers_3") (lib_id "jb_kicad:atmega_headers") (at 134.62 82.55 0) (mirror y) (unit 5)
     (in_bom yes) (on_board yes) (dnp no) (fields_autoplaced)
     (property "Reference" "J2" (at 133.3499 82.55 0)
@@
       (effects (font (size 1.27 1.27)))
     )
-    (property "Footprint" "jblocklove_kicad:arduino_mega_shield" (at 113.03 105.41 90)
+    (property "Footprint" "jb_kicad:arduino_mega_shield" (at 113.03 105.41 90)
       (effects (font (size 1.27 1.27)) hide)
     )
@@
     )
   )
-  (symbol (lib_name "atmega_headers_3") (lib_id "jblocklove_kicad:atmega_headers") (at 115.57 82.55 0) (unit 3)
+  (symbol (lib_name "atmega_headers_3") (lib_id "jb_kicad:atmega_headers") (at 115.57 82.55 0) (unit 3)
     (in_bom yes) (on_board yes) (dnp no) (fields_autoplaced)
     (property "Reference" "J2" (at 121.92 95.6032 0)
@@
       (effects (font (size 1.27 1.27)))
     )
-    (property "Footprint" "jblocklove_kicad:arduino_mega_shield" (at 137.16 105.41 90)
+    (property "Footprint" "jb_kicad:arduino_mega_shield" (at 137.16 105.41 90)
       (effects (font (size 1.27 1.27)) hide)
     )
@@
     )
   )
-  (symbol (lib_name "atmega_headers_2") (lib_id "jblocklove_kicad:atmega_headers") (at 59.055 60.325 0) (mirror y) (unit 2)
+  (symbol (lib_name "atmega_headers_2") (lib_id "jb_kicad:atmega_headers") (at 59.055 60.325 0) (mirror y) (unit 2)
     (in_bom yes) (on_board yes) (dnp no) (fields_autoplaced)
     (property "Reference" "J1" (at 59.055 59.69 0)
@@
       (effects (font (size 1.27 1.27)))
     )
-    (property "Footprint" "jblocklove_kicad:arduino_mega_shield" (at 37.465 83.185 90)
+    (property "Footprint" "jb_kicad:arduino_mega_shield" (at 37.465 83.185 90)
       (effects (font (size 1.27 1.27)) hide)
     )
@@
     )
   )
-  (symbol (lib_name "atmega_headers_3") (lib_id "jblocklove_kicad:atmega_headers") (at 133.35 57.15 0) (mirror y) (unit 6)
+  (symbol (lib_name "atmega_headers_3") (lib_id "jb_kicad:atmega_headers") (at 133.35 57.15 0) (mirror y) (unit 6)
     (in_bom yes) (on_board yes) (dnp no) (fields_autoplaced)
     (property "Reference" "J2" (at 133.3499 57.15 0)
@@
       (effects (font (size 1.27 1.27)))
     )
-    (property "Footprint" "jblocklove_kicad:arduino_mega_shield" (at 111.76 80.01 90)
+    (property "Footprint" "jb_kicad:arduino_mega_shield" (at 111.76 80.01 90)
       (effects (font (size 1.27 1.27)) hide)
     )
@@
     )
   )
-  (symbol (lib_name "atmega_headers_3") (lib_id "jblocklove_kicad:atmega_headers") (at 133.35 24.13 0) (mirror y) (unit 7)
+  (symbol (lib_name "atmega_headers_3") (lib_id "jb_kicad:atmega_headers") (at 133.35 24.13 0) (mirror y) (unit 7)
     (in_bom yes) (on_board yes) (dnp no) (fields_autoplaced)
     (property "Reference" "J2" (at 133.3499 23.495 0)
@@
       (effects (font (size 1.27 1.27)))
     )
-    (property "Footprint" "jblocklove_kicad:arduino_mega_shield" (at 111.76 46.99 90)
+    (property "Footprint" "jb_kicad:arduino_mega_shield" (at 111.76 46.99 90)
       (effects (font (size 1.27 1.27)) hide)
     )
@@
     )
   )
-  (symbol (lib_name "atmega_headers_3") (lib_id "jblocklove_kicad:atmega_headers") (at 115.57 57.15 0) (unit 2)
+  (symbol (lib_name "atmega_headers_3") (lib_id "jb_kicad:atmega_headers") (at 115.57 57.15 0) (unit 2)
     (in_bom yes) (on_board yes) (dnp no) (fields_autoplaced)
     (property "Reference" "J2" (at 121.285 70.2032 0)
@@
       (effects (font (size 1.27 1.27)))
     )
-    (property "Footprint" "jblocklove_kicad:arduino_mega_shield" (at 137.16 80.01 90)
+    (property "Footprint" "jb_kicad:arduino_mega_shield" (at 137.16 80.01 90)
       (effects (font (size 1.27 1.27)) hide)
     )
@@
     )
   )
-  (symbol (lib_name "atmega_headers_2") (lib_id "jblocklove_kicad:atmega_headers") (at 59.055 85.725 0) (mirror y) (unit 3)
+  (symbol (lib_name "atmega_headers_2") (lib_id "jb_kicad:atmega_headers") (at 59.055 85.725 0) (mirror y) (unit 3)
     (in_bom yes) (on_board yes) (dnp no) (fields_autoplaced)
     (property "Reference" "J1" (at 59.055 85.09 0)
@@
       (effects (font (size 1.27 1.27)))
     )
-    (property "Footprint" "jblocklove_kicad:arduino_mega_shield" (at 37.465 108.585 90)
+    (property "Footprint" "jb_kicad:arduino_mega_shield" (at 37.465 108.585 90)
       (effects (font (size 1.27 1.27)) hide)
     )
@@
     )
   )
-  (symbol (lib_name "atmega_headers_3") (lib_id "jblocklove_kicad:atmega_headers") (at 115.57 29.21 0) (unit 1)
+  (symbol (lib_name "atmega_headers_3") (lib_id "jb_kicad:atmega_headers") (at 115.57 29.21 0) (unit 1)
     (in_bom yes) (on_board yes) (dnp no) (fields_autoplaced)
     (property "Reference" "J2" (at 121.285 42.2632 0)
@@
       (effects (font (size 1.27 1.27)))
     )
-    (property "Footprint" "jblocklove_kicad:arduino_mega_shield" (at 137.16 52.07 90)
+    (property "Footprint" "jb_kicad:arduino_mega_shield" (at 137.16 52.07 90)
       (effects (font (size 1.27 1.27)) hide)
     )
@@
     )
   )
-  (symbol (lib_name "atmega_headers_2") (lib_id "jblocklove_kicad:atmega_headers") (at 41.275 60.325 0) (unit 6)
+  (symbol (lib_name "atmega_headers_2") (lib_id "jb_kicad:atmega_headers") (at 41.275 60.325 0) (unit 6)
     (in_bom yes) (on_board yes) (dnp no) (fields_autoplaced)
     (property "Reference" "J1" (at 46.355 73.3782 0)
@@
       (effects (font (size 1.27 1.27)))
     )
-    (property "Footprint" "jblocklove_kicad:arduino_mega_shield" (at 62.865 83.185 90)
+    (property "Footprint" "jb_kicad:arduino_mega_shield" (at 62.865 83.185 90)
       (effects (font (size 1.27 1.27)) hide)
     )
