File: kicad/offramps/fet_bidir_level_shifters.kicad_sch (KiCad schematic)
At the start: 6 parts, among them Q3 BSS138, Q4 BSS138

Commit message: Power side channel analysis largely done. Lots of cleanup and odds-and-ends. On-schematic notes for what's left as of this commit.
Parts:
- renumbered Q3 to Q13, Q4 to Q14, R15 to R3, R16 to R31, R17 to R32, R18 to R33
Connections:
- net 3p3V_sel renamed +3V3_sel
- net 5V_sel renamed +++5V_sel
Changed lines of the file:
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@@
 		(dnp no)
 		(fields_autoplaced yes)
-		(property "Reference" "R15"
+		(property "Reference" "R3"
 			(at 40.64 34.2899 0)
 			(effects
@@
 		(instances
 			(project "offramps"
-				(path "/e859ad58-cc0a-46d6-9578-387f2d0c634f/20b9d5f0-f1f3-4dff-9e31-c0e7967226ea"
-					(reference "R15")
-					(unit 1)
-				)
 				(path "/e859ad58-cc0a-46d6-9578-387f2d0c634f/9ea056cf-6c8f-4797-81ba-dbc6d64757ab"
 					(reference "R3")
@@
 		(dnp no)
 		(fields_autoplaced yes)
-		(property "Reference" "R17"
+		(property "Reference" "R32"
 			(at 58.42 34.2899 0)
 			(effects
@@
 		(instances
 			(project "offramps"
-				(path "/e859ad58-cc0a-46d6-9578-387f2d0c634f/20b9d5f0-f1f3-4dff-9e31-c0e7967226ea"
-					(reference "R17")
-					(unit 1)
-				)
 				(path "/e859ad58-cc0a-46d6-9578-387f2d0c634f/9ea056cf-6c8f-4797-81ba-dbc6d64757ab"
 					(reference "R32")
@@
 		(dnp no)
 		(fields_autoplaced yes)
-		(property "Reference" "Q4"
+		(property "Reference" "Q14"
 			(at 46.99 80.01 90)
 			(effects
@@
 		(instances
 			(project "offramps"
-				(path "/e859ad58-cc0a-46d6-9578-387f2d0c634f/20b9d5f0-f1f3-4dff-9e31-c0e7967226ea"
-					(reference "Q4")
-					(unit 1)
-				)
 				(path "/e859ad58-cc0a-46d6-9578-387f2d0c634f/9ea056cf-6c8f-4797-81ba-dbc6d64757ab"
 					(reference "Q14")
@@
 		(dnp no)
 		(fields_autoplaced yes)
-		(property "Reference" "#PWR034"
+		(property "Reference" "#PWR054"
 			(at 55.88 60.96 0)
 			(effects
@@
 			)
 		)
-		(property "Value" "5V_sel"
+		(property "Value" "+++5V_sel"
 			(at 55.88 52.07 0)
 			(effects
@@
 		(instances
 			(project "offramps"
-				(path "/e859ad58-cc0a-46d6-9578-387f2d0c634f/20b9d5f0-f1f3-4dff-9e31-c0e7967226ea"
-					(reference "#PWR034")
-					(unit 1)
-				)
 				(path "/e859ad58-cc0a-46d6-9578-387f2d0c634f/9ea056cf-6c8f-4797-81ba-dbc6d64757ab"
 					(reference "#PWR054")
@@
 		(dnp no)
 		(fields_autoplaced yes)
-		(property "Reference" "R18"
+		(property "Reference" "R33"
 			(at 58.42 66.0399 0)
 			(effects
@@
 		(instances
 			(project "offramps"
-				(path "/e859ad58-cc0a-46d6-9578-387f2d0c634f/20b9d5f0-f1f3-4dff-9e31-c0e7967226ea"
-					(reference "R18")
-					(unit 1)
-				)
 				(path "/e859ad58-cc0a-46d6-9578-387f2d0c634f/9ea056cf-6c8f-4797-81ba-dbc6d64757ab"
 					(reference "R33")
@@
 		(dnp no)
 		(fields_autoplaced yes)
-		(property "Reference" "Q3"
+		(property "Reference" "Q13"
 			(at 46.99 48.26 90)
 			(effects
@@
 		(instances
 			(project "offramps"
-				(path "/e859ad58-cc0a-46d6-9578-387f2d0c634f/20b9d5f0-f1f3-4dff-9e31-c0e7967226ea"
-					(reference "Q3")
-					(unit 1)
-				)
 				(path "/e859ad58-cc0a-46d6-9578-387f2d0c634f/9ea056cf-6c8f-4797-81ba-dbc6d64757ab"
 					(reference "Q13")
@@
 		(dnp no)
 		(fields_autoplaced yes)
-		(property "Reference" "R16"
+		(property "Reference" "R31"
 			(at 40.64 66.0399 0)
 			(effects
@@
 		(instances
 			(project "offramps"
-				(path "/e859ad58-cc0a-46d6-9578-387f2d0c634f/20b9d5f0-f1f3-4dff-9e31-c0e7967226ea"
-					(reference "R16")
-					(unit 1)
-				)
 				(path "/e859ad58-cc0a-46d6-9578-387f2d0c634f/9ea056cf-6c8f-4797-81ba-dbc6d64757ab"
 					(reference "R31")
@@
 		(dnp no)
 		(fields_autoplaced yes)
-		(property "Reference" "#PWR032"
+		(property "Reference" "#PWR07"
 			(at 38.1 60.96 0)
 			(effects
@@
 			)
 		)
-		(property "Value" "3p3V_sel"
+		(property "Value" "+3V3_sel"
 			(at 38.1 52.07 0)
 			(effects
@@
 		(instances
 			(project "offramps"
-				(path "/e859ad58-cc0a-46d6-9578-387f2d0c634f/20b9d5f0-f1f3-4dff-9e31-c0e7967226ea"
-					(reference "#PWR032")
-					(unit 1)
-				)
 				(path "/e859ad58-cc0a-46d6-9578-387f2d0c634f/9ea056cf-6c8f-4797-81ba-dbc6d64757ab"
 					(reference "#PWR07")
@@
 		(dnp no)
 		(fields_autoplaced yes)
-		(property "Reference" "#PWR033"
+		(property "Reference" "#PWR08"
 			(at 55.88 29.21 0)
 			(effects
@@
 			)
 		)
-		(property "Value" "5V_sel"
+		(property "Value" "+++5V_sel"
 			(at 55.88 20.32 0)
 			(effects
@@
 		(instances
 			(project "offramps"
-				(path "/e859ad58-cc0a-46d6-9578-387f2d0c634f/20b9d5f0-f1f3-4dff-9e31-c0e7967226ea"
-					(reference "#PWR033")
-					(unit 1)
-				)
 				(path "/e859ad58-cc0a-46d6-9578-387f2d0c634f/9ea056cf-6c8f-4797-81ba-dbc6d64757ab"
 					(reference "#PWR08")
@@
 		(dnp no)
 		(fields_autoplaced yes)
-		(property "Reference" "#PWR031"
+		(property "Reference" "#PWR05"
 			(at 38.1 29.21 0)
 			(effects
@@
 			)
 		)
-		(property "Value" "3p3V_sel"
+		(property "Value" "+3V3_sel"
 			(at 38.1 20.32 0)
 			(effects
@@
 		(instances
 			(project "offramps"
-				(path "/e859ad58-cc0a-46d6-9578-387f2d0c634f/20b9d5f0-f1f3-4dff-9e31-c0e7967226ea"
-					(reference "#PWR031")
-					(unit 1)
-				)
 				(path "/e859ad58-cc0a-46d6-9578-387f2d0c634f/9ea056cf-6c8f-4797-81ba-dbc6d64757ab"
 					(reference "#PWR05")
