File: kicad/offramps/offramps.kicad_sch (KiCad schematic)
At the start: 126 parts, among them J10 Conn_Coaxial, J11 Conn_Coaxial, J12 Conn_Coaxial, J13 Conn_01x04, J15 Micro_SD_Card, J3 ASP-134606-01, J4 Conn_01x04_Pin, J5 Screw_Terminal_01x02, J6 Conn_01x03_Male, J7 Screw_Terminal_01x02, J8 Conn_01x06_Male, J9 Conn_Coaxial, Q10 BSS138, Q5 BSS138, Q6 BSS138, Q7 BSS138, Q8 BSS138, Q9 BSS138, U1 AMS1117-3.3, U10 PTMUX4053PWR, U11 LIS2MDLTR, U12 LIS2MDLTR, U13 ADS1115IDGS, U15 ADC1173CIMTC/NOPB, U16 ADS1114IDGS, U2 TXB0108PWR, U3 TXB0108PWR, U4 TXB0108PWR, U5 TXB0108PWR, U6 TXB0108PWR, U7 LSM6DSRTR, U8 MCP4725xxx-xCH, U9 MCP4725xxx-xCH

Commit message: Power side channel analysis largely done. Lots of cleanup and odds-and-ends. On-schematic notes for what's left as of this commit.
Parts:
- removed J13: Conn_01x04, Connector_PinSocket_2.54mm:PinSocket_1x04_P2.54mm_Vertical, symbol Connector_Generic:Conn_01x04
- removed R40: 100k, Resistor_SMD:R_0805_2012Metric, symbol Device:R
- removed R41, R42, R43, R44: 16k, Resistor_SMD:R_0805_2012Metric, symbol Device:R
- removed R45: 0, Resistor_SMD:R_0805_2012Metric, symbol Device:R
- removed U12: LIS2MDLTR, Package_LGA:LGA-12_2x2mm_P0.5mm, symbol kiwih_kicad:LIS2MDLTR
- removed U13: ADS1115IDGS, Package_SO:TSSOP-10_3x3mm_P0.5mm, symbol Analog_ADC:ADS1115IDGS
- removed U15: ADC1173CIMTC/NOPB, MTC24, symbol ADC1173:ADC1173CIMTC_NOPB
- added C28, C29, C32: 100n, symbol Device:C
- added C31: 2.2u, symbol Device:C
- added J14: Conn_Coaxial, symbol Connector:Conn_Coaxial
- added J16: Conn_01x03_Male, Connector_PinHeader_2.54mm:PinHeader_1x03_P2.54mm_Vertical, symbol Connector:Conn_01x03_Male
- added L1: 10u, symbol Device:L
- added Q1, Q11, Q12, Q2, Q3, Q4: BSS138, Package_TO_SOT_SMD:SOT-23, symbol Transistor_FET:BSS138
- added R12, R13, R14, R15, R16, R17, R18, R27, R28, R29, R3, R6: 10k, symbol Device:R
- added R30: 27, symbol Device:R
- added R31: 270, symbol Device:R
- added R32: 4.7k, Resistor_SMD:R_0805_2012Metric, symbol Device:R
- added R33: 10K, Resistor_SMD:R_0805_2012Metric, symbol Device:R
- added R50: 10R, symbol Device:R
- added U12: LMH6611MK/NOPB, MK06A, symbol offramps_lib:LMH6611MK_NOPB
- added U13: TXB0108PWR, external_footprints:SOP65P640X120-20N, symbol TXB0108PWR:TXB0108PWR
- added U14: ADC1175CIMTC/NOPB, MTC24_TEX, symbol offramps_lib:ADC1175CIMTC_NOPB
- C22: value 10uF -> 100n
- C23: value 100nF -> 1uF; Vendor C49678 -> C28323
- C24: value 100nF -> 100n; footprint Capacitor_SMD:C_0805_2012Metric -> (none); Vendor C49678 -> (none)
- C25: value 220nF -> 100n; footprint Capacitor_SMD:C_0805_2012Metric -> (none); Vendor C5378 -> (none)
- C26: value 100n -> C; footprint Capacitor_SMD:C_0805_2012Metric -> (none); Vendor C49678 -> (none); now not fitted
- C27: value 1uF -> 2.2u; footprint Capacitor_SMD:C_0805_2012Metric -> (none); Vendor C28323 -> (none)
- R19: value 10k -> 25
- R20: value 10k -> 110
- R37, R38, R39: value 100k -> 10K; Vendor C17407 -> C17414
- R46, R47, R48, R49: now not fitted
Connections:
- net 3p3V_sel is gone; now on net +3V3_sel: C10.1, C15.1, C16.1, C3.1, C30.1, C4.1, C7.1, C9.1, J15.4 (VDD), J2.4 (+3V3), J4.2 (Pin_2), Q10.2 (S), Q5.2 (S), Q6.2 (S), Q7.2 (S), Q8.2 (S), Q9.2 (S), R1.1, R19.1, R2.1, R34.1, R4.1, R46.1, R47.1, R48.1, R49.1, R5.1, U2.10 (OE), U2.2 (VCCA), U3.10 (OE), U3.2 (VCCA), U4.10 (OE), U4.2 (VCCA), U5.10 (OE), U5.2 (VCCA), U6.10 (OE), U6.2 (VCCA), U8.3 (VDD), U8.6 (A0), U9.3 (VDD)
- net 5V_sel is gone; now on net +5V_sel: C11.1, C12.1, C17.1, C5.1, C6.1, C8.1, J2.5 (+5V), J2.59 (+5V), J2.60 (+5V), J6.2 (Pin_2), J8.1 (Pin_1), R20.1, U10.16 (VDD), U2.19 (VCCB), U3.19 (VCCB), U4.19 (VCCB), U5.19 (VCCB), U6.19 (VCCB)
- net AIN0 is gone; now on net fpga_SDA: R37.2
- net AIN0_DIV is gone; now on net +3V3_sel: R37.1
- net AIN1 is gone; now on net fpga_SCL: R38.2
- net AIN1_DIV is gone; now on net +3V3_sel: R38.1
- net AIN2 is gone; now on net fpga_SDA: R39.2
- net AIN2_DIV is gone; now on net +3V3_sel: R39.1
- net SPI_MON_IMU_CS is gone; now on net +3V3_sel: U7.12 (CS)
- net SPI_MON_MOSI is gone; now on net fpga_SDA: U7.14 (SDA)
- net SPI_MON_SCK is gone; now on net fpga_SCL: U7.13 (SCL)
- net f_ls_D10: now also J3.G24 (LA22_P)
- net f_ls_D8: now also J3.G27 (LA25_P)
- net f_ls_D9: now also J3.G25 (LA22_N)
- net f_ls_E0-DIR: now also J3.G22 (LA20_N)
- net f_ls_E0-EN: now also J3.G12 (LA08_P)
- net f_ls_E0-STEP: now also J3.G21 (LA20_P)
- net f_ls_E1-DIR: now also J3.G10 (LA03_N), Q2.2 (S), R6.2
- net f_ls_E1-EN: now also J3.G13 (LA08_N)
- net f_ls_E1-STEP: now also J3.G09 (LA03_P), Q1.2 (S), R3.2
- net f_ls_UART_RX: now also J3.D14 (LA09_P), Q4.3 (D), R17.2
- net f_ls_UART_TX: now also J3.D11 (LA05_P), Q11.2 (S), R18.2
- net f_ls_X-DIR: now also J3.G30 (LA29_P)
- net f_ls_X-EN: now also J3.G31 (LA29_N)
- net f_ls_X-MAX: now also J3.H32 (LA28_N)
- net f_ls_X-MIN: now also J3.H31 (LA28_P)
- net f_ls_X-STEP: now also J3.G28 (LA25_N)
- net f_ls_Y-DIR: now also J3.G16 (LA12_N)
- net f_ls_Y-EN: now also J3.G33 (LA31_P)
- net f_ls_Y-MAX: now also J3.H35 (LA30_N)
- net f_ls_Y-MIN: now also J3.H34 (LA30_P)
- net f_ls_Y-STEP: now also J3.G15 (LA12_P)
- net f_ls_Z-DIR: now also J3.G19 (LA16_N)
- net f_ls_Z-EN: now also J3.G34 (LA31_N)
- net f_ls_Z-MAX: now also J3.H38 (LA32_N)
- net f_ls_Z-MIN: now also J3.H37 (LA32_P)
- net f_ls_Z-STEP: now also J3.G18 (LA16_P)
- net f_sd_cmd: now also J3.C18 (LA14_P)
- net f_sd_dat0: now also J3.C14 (LA10_P)
- net f_sd_dat1: now also J3.C15 (LA10_N)
- net f_sd_dat2: now also J3.C10 (LA06_P)
- net f_sd_dat3: now also J3.C11 (LA06_N)
- net ls_f_D10: now also J3.H07 (LA02_P)
- net ls_f_D8: now also J3.H10 (LA04_P)
- net ls_f_D9: now also J3.H08 (LA02_N)
- net ls_f_E0-DIR: now also J3.H29 (LA24_N)
- net ls_f_E0-EN: now also J3.H19 (LA15_P)
- net ls_f_E0-STEP: now also J3.H28 (LA24_P)
- net ls_f_E1-DIR: now also J3.G36 (LA33_P), U4.1 (A1)
- net ls_f_E1-EN: now also J3.H20 (LA15_N)
- net ls_f_E1-STEP: now also J3.G37 (LA33_N), U4.3 (A2)
- net ls_f_UART_RX: now also J3.D12 (LA05_N), Q12.2 (S), R28.2
- net ls_f_UART_TX: now also J3.D15 (LA09_N), Q3.3 (D), R15.2
- net ls_f_X-DIR: now also J3.H13 (LA07_P)
- net ls_f_X-EN: now also J3.H14 (LA07_N)
- net ls_f_X-MAX: now also J3.C26 (LA27_P)
- net ls_f_X-MIN: now also J3.C19 (LA14_N)
- net ls_f_X-STEP: now also J3.H11 (LA04_N)
- net ls_f_Y-DIR: now also J3.H23 (LA19_N)
- net ls_f_Y-EN: now also J3.H16 (LA11_P)
- net ls_f_Y-MAX: now also J3.C27 (LA27_N)
- net ls_f_Y-MIN: now also J3.C22 (LA18_P_CC)
- net ls_f_Y-STEP: now also J3.H22 (LA19_P)
- net ls_f_Z-DIR: now also J3.H26 (LA21_N)
- net ls_f_Z-EN: now also J3.H17 (LA11_N)
- net ls_f_Z-MAX: now also J3.D17 (LA13_P)
- net ls_f_Z-MIN: now also J3.C23 (LA18_N_CC)
- net ls_f_Z-STEP: now also J3.H25 (LA21_P)
- net ls_jump_E1-DIR: now also Q2.3 (D), R13.2
- net ls_jump_E1-STEP: now also Q1.3 (D), R12.2
- net ls_jump_UART_RX: now also Q4.2 (S), R16.2
- net ls_jump_UART_TX: now also Q11.3 (D), R27.2
- net r_UART_TX: now also Q12.3 (D), R29.2
- net u_E1-DIR: now also U4.20 (B1)
- net u_E1-STEP: now also U4.18 (B2)
- net u_UART_TX: now also Q3.2 (S), R14.2
- net +5V_sel: now reaches C25.1
- net +5V_sel: now also L1.1, R12.1, R13.1, R15.1, R17.1, R27.1, R29.1
- net +3V3_sel: now reaches U11.6 (INT/DRDY/SDO)
- net +3V3_sel: now also C1.2, C10.2, C11.2, C12.2, C13.1, C13.2, C14.1, C14.2, C15.2, C16.2, C17.2, C18.1, C18.2, C19.1, C19.2, C2.2, C20.1, C20.2, C21.2, C22.1, C22.2, C23.1, C23.2, C24.2, C26.2, C27.2, C3.2, C30.2, C4.2, C5.2, C6.2, C7.2, C8.2, C9.2, D1.1 (K), D2.1 (K), J1.25 (GND), J1.26 (GND), J1.6 (GND), J1.7 (GND), J1.83 (GND), J10.2 (Ext), J15.6 (VSS), J15.9 (SHIELD), J2.25 (GND), J2.26 (GND), J2.6 (GND), J2.7 (GND), J2.83 (GND), J3.C01 (GND), J3.C04 (GND), J3.C05 (GND), J3.C08 (GND), J3.C09 (GND), J3.C12 (GND), J3.C13 (GND), J3.C16 (GND), J3.C17 (GND), J3.C20 (GND), J3.C21 (GND), J3.C24 (GND), J3.C25 (GND), J3.C28 (GND), J3.C29 (GND), J3.C32 (GND), J3.C33 (GND), J3.C36 (GND), J3.C38 (GND), J3.C40 (GND), J3.D02 (GND), J3.D03 (GND), J3.D06 (GND), J3.D07 (GND), J3.D10 (GND), J3.D13 (GND), J3.D16 (GND), J3.D19 (GND), J3.D22 (GND), J3.D25 (GND), J3.D28 (GND), J3.D37 (GND), J3.D39 (GND), J3.G01 (GND), J3.G04 (GND), J3.G05 (GND), J3.G08 (GND), J3.G11 (GND), J3.G14 (GND), J3.G17 (GND), J3.G20 (GND), J3.G23 (GND), J3.G26 (GND), J3.G29 (GND), J3.G32 (GND), J3.G35 (GND), J3.G38 (GND), J3.G40 (GND), J3.H03 (GND), J3.H06 (GND), J3.H09 (GND), J3.H12 (GND), J3.H15 (GND), J3.H18 (GND), J3.H21 (GND), J3.H24 (GND), J3.H27 (GND), J3.H30 (GND), J3.H33 (GND), J3.H36 (GND), J3.H39 (GND), J5.2 (Pin_2), J7.2 (Pin_2), J8.6 (Pin_6), J9.2 (Ext), R1.2, R11.2, R2.2, R21.2, R22.2, R23.2, R24.2, R25.2, R26.2, R34.2, R35.1, R36.1, R4.2, R5.2, R7.2, R9.2, U1.1 (GND), U10.6 (*EN), U10.7 (VSS), U10.8 (GND), U11.10 (VDD_IO), U11.3 (~{CS}), U11.8 (GND), U11.9 (VDD), U16.1 (ADDR), U16.3 (GND), U16.8 (VDD), U2.11 (GND), U3.11 (GND), U4.11 (GND), U5.11 (GND), U6.11 (GND), U7.2 (SDX), U7.3 (SCX), U7.5 (VDDIO), U7.6 (GND), U7.7 (GND), U7.8 (VDD), U8.2 (VSS), U9.2 (VSS), U9.6 (A0), C28.2, C29.2, C31.2, C32.2, J14.2 (Ext), Q1.1 (G), Q11.1 (G), Q12.1 (G), Q2.1 (G), Q3.1 (G), Q4.1 (G), R14.1, R16.1, R18.1, R28.1, R3.1, R32.1, R33.1, R6.1, U12.2 (V-), U12.3 (IN+), U13.11 (GND), U13.2 (VCCA), U14.2 (DVSS), U14.20 (AVSS), U14.21 (AVSS), U14.24 (DVSS)
- net fpga_SCL: now reaches J3.C30 (SCL)
- net fpga_SCL: now also R35.2, U11.1 (SCL/SPC), U16.10 (SCL), R33.2
- net fpga_SDA: now reaches J3.C31 (SDA)
- net fpga_SDA: now also R36.2, U11.4 (SDA/SDI/SDO), U16.9 (SDA)
- removed net +3V3: C13.1, C14.1, C18.1, C19.1, C20.1, C22.1, C23.1, C24.1, C26.2, C27.2, R35.1, R36.1, U11.10 (VDD_IO), U11.3 (~{CS}), U11.9 (VDD), U7.5 (VDDIO), U7.8 (VDD)
- net 3p3V_DC_in renamed +3V3_DC_in
- net 3p3V_reg renamed +3V3_reg
- net 3p3V_uC renamed +3V3_uC
- net 5V_uC renamed +5V_uC
- net 5v_DC_in renamed +5V_DC_in
- removed net GND: C1.2, C10.2, C11.2, C12.2, C13.2, C14.2, C15.2, C16.2, C17.2, C18.2, C19.2, C2.2, C20.2, C21.2, C22.2, C23.2, C24.2, C25.2, C26.1, C27.1, C3.2, C30.2, C4.2, C5.2, C6.2, C7.2, C8.2, C9.2, D1.1 (K), D2.1 (K), J1.25 (GND), J1.26 (GND), J1.6 (GND), J1.7 (GND), J1.83 (GND), J10.2 (Ext), J15.6 (VSS), J15.9 (SHIELD), J2.25 (GND), J2.26 (GND), J2.6 (GND), J2.7 (GND), J2.83 (GND), J3.C01 (GND), J3.C04 (GND), J3.C05 (GND), J3.C08 (GND), J3.C09 (GND), J3.C12 (GND), J3.C13 (GND), J3.C16 (GND), J3.C17 (GND), J3.C20 (GND), J3.C21 (GND), J3.C24 (GND), J3.C25 (GND), J3.C28 (GND), J3.C29 (GND), J3.C32 (GND), J3.C33 (GND), J3.C36 (GND), J3.C38 (GND), J3.C40 (GND), J3.D02 (GND), J3.D03 (GND), J3.D06 (GND), J3.D07 (GND), J3.D10 (GND), J3.D13 (GND), J3.D16 (GND), J3.D19 (GND), J3.D22 (GND), J3.D25 (GND), J3.D28 (GND), J3.D37 (GND), J3.D39 (GND), J3.G01 (GND), J3.G04 (GND), J3.G05 (GND), J3.G08 (GND), J3.G11 (GND), J3.G14 (GND), J3.G17 (GND), J3.G20 (GND), J3.G23 (GND), J3.G26 (GND), J3.G29 (GND), J3.G32 (GND), J3.G35 (GND), J3.G38 (GND), J3.G40 (GND), J3.H03 (GND), J3.H06 (GND), J3.H09 (GND), J3.H12 (GND), J3.H15 (GND), J3.H18 (GND), J3.H21 (GND), J3.H24 (GND), J3.H27 (GND), J3.H30 (GND), J3.H33 (GND), J3.H36 (GND), J3.H39 (GND), J5.2 (Pin_2), J7.2 (Pin_2), J8.6 (Pin_6), J9.2 (Ext), R1.2, R11.2, R2.2, R21.2, R22.2, R23.2, R24.2, R25.2, R26.2, R34.2, R4.2, R5.2, R7.2, R9.2, U1.1 (GND), U10.6 (*EN), U10.7 (VSS), U10.8 (GND), U11.6 (INT/DRDY/SDO), U11.8 (GND), U2.11 (GND), U3.11 (GND), U4.11 (GND), U5.11 (GND), U6.11 (GND), U7.6 (GND), U7.7 (GND), U8.2 (VSS), U9.2 (VSS), U9.6 (A0)
- removed net IMU_I2C_SCL: R36.2, U11.1 (SCL/SPC), U7.3 (SCX)
- removed net IMU_I2C_SDA: R35.2, U11.4 (SDA/SDI/SDO), U7.2 (SDX)
- net SPI_MON_MISO: no longer names the net of U7.1 (SDO/SA0)
- new net: J16.2 (Pin_2), U14.12 (CLK)
- new net: L1.2, R50.2
- new net: R30.2, R31.1, U12.4 (IN-)
- new net: C25.2, R30.1
- new net: R32.2, U13.10 (OE)
- new net: U13.12 (B8), U14.10 (D7)
- new net: U13.13 (B7), U14.9 (D6)
- new net: U13.14 (B6), U14.8 (D5)
- new net: U13.15 (B5), U14.7 (D4)
- new net: U13.16 (B4), U14.6 (D3)
- new net: U13.17 (B3), U14.5 (D2)
- new net: U13.18 (B2), U14.4 (D1)
- new net: U13.20 (B1), U14.3 (D0)
- new net +5V_filt: C24.1, C27.1, C28.1, C29.1, C31.1, C32.1, R50.1, U12.5 (~DIS), U12.6 (V+), U13.19 (VCCB), U14.11 (DVDD), U14.13 (DVDD), U14.14 (AVDD), U14.15 (AVDD), U14.18 (AVDD)
- new net ext_scope_clk: J14.1 (In), J16.3 (Pin_3)
- new net f_psc_ain: C26.1, R31.2, U12.1 (OUT), U14.19 (VIN)
- new net f_scope_clk: J16.1 (Pin_1)
- new net psc_d0: U13.1 (A1)
- new net psc_d1: U13.3 (A2)
- new net psc_d2: U13.4 (A3)
- new net psc_d3: U13.5 (A4)
- new net psc_d4: U13.6 (A5)
- new net psc_d5: U13.7 (A6)
- new net psc_d6: U13.8 (A7)
- new net psc_d7: U13.9 (A8)
- no-connect marks 16 -> 13
Other:
- removed sheet f_r_E1_SHIFTER
- removed sheet f_r_UART_SHIFTER
- removed sheet u_f_E1_SHIFTER
- removed sheet u_f_UART_SHIFTER
- note added: "+5V can be pulled from the Ardiuno or a screw terminal"
- note added: "0-5V input become 0-3V3 Voltage divider (R2)/(R1+R2) = 1/3 = R2 = 5K, R1 = 10K"
- note added: "3.3V can be pulled from the Ardiuno, a screw terminal, or a voltage regulator from the +5V"
- note added: "ADCs"
- note added: "ADD VOLTAGE FOLLOWERS?"
- note added: "CHECK"
- note added: "CW Nano schematic and documentation reference have notable differences..."
- note added: "DACs"
- note added: "FPGA -> RAMPS Level Shifters"
- note added: "Power analysis clock selection"
- note added: "Thermistor Muxltiplexing"
- note added: "VGND?"
- note added: "uC -> FPGA Level Shifters"
- note removed: "0-24V input become 0-3V3 about a factor of 7.5 voltage divider (R2)/(R1+R2) = 1/6 = R2 = 100K, R1 = 16K"
- note removed: "ADC (Inputs)"
- note removed: "ADD VOLTAGE FOLLOWERS"
- note removed: "AIN0 and AIN1 swapped on chip for routing reasons"
- note removed: "COMBINE"
- note removed: "FIX"
- note removed: "FPGA -> RAMPS Side Shifters"
- note removed: "NOTES"
- note removed: "SET THIS UP"
- note removed: "THINGS TO DO: - 5V LED - 12V LED? - 12V Connection to Mezz?"
- note removed: "Thermistor ADCs"
- note removed: "Thermistor DACs"
- note removed: "Thermistor Mux"
- note removed: "uC -> FPGA Side Shifters"
- moved on the sheet: C1, C10, C11, C12, C13, C14, C15, C16, C17, C18, C19, C2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
