File: kicad/offramps/offramps.kicad_sch (KiCad schematic)
At the start: 149 parts, among them J10 Conn_Coaxial, J11 Conn_Coaxial, J12 Conn_Coaxial, J14 Conn_Coaxial, J15 Micro_SD_Card, J16 Conn_01x03_Male, J3 ASP-134606-01, J4 Conn_01x04_Pin, J5 Screw_Terminal_01x02, J6 Conn_01x03_Male, J7 Screw_Terminal_01x02, J8 Conn_01x06_Male, J9 Conn_Coaxial, Q1 BSS138, Q10 BSS138, Q11 BSS138, Q12 BSS138, Q2 BSS138, Q3 BSS138, Q4 BSS138, Q5 BSS138, Q6 BSS138, Q7 BSS138, Q8 BSS138, Q9 BSS138, U1 AMS1117-3.3, U10 PTMUX4053PWR, U11 LIS2MDLTR, U12 LMH6611MK/NOPB, U13 TXB0108PWR, U14 ADC1175CIMTC/NOPB, U16 ADS1114IDGS, U2 TXB0108PWR, U3 TXB0108PWR, U4 TXB0108PWR, U5 TXB0108PWR, U6 TXB0108PWR, U7 LSM6DSRTR, U8 MCP4725xxx-xCH, U9 MCP4725xxx-xCH

Commit message: Major changes and updates. Hopefully mostly done. Need to check/finish the ADC setup and finish some other cleanup. Need to finish populating the FMC
Parts:
- removed J3: ASP-134606-01, SAMTEC_ASP-134606-01, symbol ASP-134606-01:ASP-134606-01
- removed TP1: TestPoint_Flag, symbol Connector:TestPoint_Flag
- removed TP2: TestPoint, symbol Connector:TestPoint
- added C33, C34, C35, C36, C40, C41, C42: 100n, symbol Device:C
- added C37: C, symbol Device:C
- added C38, C39: 2.2u, symbol Device:C
- added J13: VITA_57.1_FMC_HPC_Carrier, Connector_Samtec:Samtec_FMC_ASP-134486-01_10x40_P1.27mm_Vertical, symbol jblocklove_libs:VITA_57.1_FMC_HPC_Carrier
- added J3: Conn_01x02_Pin, symbol Connector:Conn_01x02_Pin
- added Q13, Q14, Q15, Q16: NPN, symbol Simulation_SPICE:NPN
- added R40: 27, symbol Device:R
- added R41: 270, symbol Device:R
- added R42, R56, R57, R58, R59, R60, R61, R62, R63: 10k, symbol Device:R
- added R43, R44, R45, R51, R52, R53, R54, R55: 100, symbol Device:R
- added SW1: SW_DIP_x08, symbol Switch:SW_DIP_x08
- added TP1, TP2, TP3, TP4, TP5: TestPoint_Probe, symbol Connector:TestPoint_Probe
- added U15: LMH6611MK/NOPB, MK06A, symbol offramps_lib:LMH6611MK_NOPB
- added U17: POPA2994IDGKR, VSSOP8_DGK_TEX, symbol offramps_lib:POPA2994IDGKR
- added U18: ADC1173CIMTC/NOPB, MTC24, symbol offramps_lib:ADC1173CIMTC_NOPB
- added U19: LTC-4627JR, Display_7Segment:LTC-4627Jx, symbol Display_Character:LTC-4627JR
- R10, R8: footprint Resistor_SMD:R_0805_2012Metric -> (none); Vendor C2828783 -> (none)
- R11, R9: footprint Resistor_SMD:R_0805_2012Metric -> (none); Vendor C17414 -> (none)
- R19: value 25 -> 100
- R20: value 110 -> 470
- renumbered TP3 to TP?
Connections:
- net +3V3_sel: now also R11.1, R9.1, C34.1, C35.1, C36.2, C37.2, C38.2, C39.2, C40.2, C41.2, C42.2, J13.A1 (GND), J13.A12 (GND), J13.A13 (GND), J13.A16 (GND), J13.A17 (GND), J13.A20 (GND), J13.A21 (GND), J13.A24 (GND), J13.A25 (GND), J13.A28 (GND), J13.A29 (GND), J13.A32 (GND), J13.A33 (GND), J13.A36 (GND), J13.A37 (GND), J13.A4 (GND), J13.A40 (GND), J13.A5 (GND), J13.A8 (GND), J13.A9 (GND), J13.B10 (GND), J13.B11 (GND), J13.B14 (GND), J13.B15 (GND), J13.B18 (GND), J13.B19 (GND), J13.B2 (GND), J13.B22 (GND), J13.B23 (GND), J13.B26 (GND), J13.B27 (GND), J13.B3 (GND), J13.B30 (GND), J13.B31 (GND), J13.B34 (GND), J13.B35 (GND), J13.B38 (GND), J13.B39 (GND), J13.B6 (GND), J13.B7 (GND), J13.C1 (GND), J13.C12 (GND), J13.C13 (GND), J13.C16 (GND), J13.C17 (GND), J13.C20 (GND), J13.C21 (GND), J13.C24 (GND), J13.C25 (GND), J13.C28 (GND), J13.C29 (GND), J13.C32 (GND), J13.C33 (GND), J13.C36 (GND), J13.C38 (GND), J13.C4 (GND), J13.C40 (GND), J13.C5 (GND), J13.C8 (GND), J13.C9 (GND), J13.D10 (GND), J13.D13 (GND), J13.D16 (GND), J13.D19 (GND), J13.D2 (GND), J13.D22 (GND), J13.D25 (GND), J13.D28 (GND), J13.D3 (GND), J13.D37 (GND), J13.D39 (GND), J13.D6 (GND), J13.D7 (GND), J13.E1 (GND), J13.E11 (GND), J13.E14 (GND), J13.E17 (GND), J13.E20 (GND), J13.E23 (GND), J13.E26 (GND), J13.E29 (GND), J13.E32 (GND), J13.E35 (GND), J13.E38 (GND), J13.E4 (GND), J13.E40 (GND), J13.E5 (GND), J13.E8 (GND), J13.F12 (GND), J13.F15 (GND), J13.F18 (GND), J13.F2 (GND), J13.F21 (GND), J13.F24 (GND), J13.F27 (GND), J13.F3 (GND), J13.F30 (GND), J13.F33 (GND), J13.F36 (GND), J13.F39 (GND), J13.F6 (GND), J13.F9 (GND), J13.G1 (GND), J13.G11 (GND), J13.G14 (GND), J13.G17 (GND), J13.G20 (GND), J13.G23 (GND), J13.G26 (GND), J13.G29 (GND), J13.G32 (GND), J13.G35 (GND), J13.G38 (GND), J13.G4 (GND), J13.G40 (GND), J13.G5 (GND), J13.G8 (GND), J13.H12 (GND), J13.H15 (GND), J13.H18 (GND), J13.H21 (GND), J13.H24 (GND), J13.H27 (GND), J13.H3 (GND), J13.H30 (GND), J13.H33 (GND), J13.H36 (GND), J13.H39 (GND), J13.H6 (GND), J13.H9 (GND), J13.J1 (GND), J13.J11 (GND), J13.J14 (GND), J13.J17 (GND), J13.J20 (GND), J13.J23 (GND), J13.J26 (GND), J13.J29 (GND), J13.J32 (GND), J13.J35 (GND), J13.J38 (GND), J13.J4 (GND), J13.J40 (GND), J13.J5 (GND), J13.J8 (GND), J13.K12 (GND), J13.K15 (GND), J13.K18 (GND), J13.K2 (GND), J13.K21 (GND), J13.K24 (GND), J13.K27 (GND), J13.K3 (GND), J13.K30 (GND), J13.K33 (GND), J13.K36 (GND), J13.K39 (GND), J13.K6 (GND), J13.K9 (GND), J3.2 (Pin_2), Q13.3 (E), Q14.3 (E), Q15.3 (E), Q16.3 (E), R42.1, R56.1, R57.1, R58.1, R59.1, R60.1, R61.1, R62.1, R63.1, SW1.10, SW1.11, SW1.12, SW1.13, SW1.14, SW1.15, SW1.16, SW1.9, TP1.1, TP2.1, TP3.1, TP4.1, TP5.1, U15.2 (V-), U15.3 (IN+), U17.4 (V-), U18.2 (DVSS), U18.20 (AVSS), U18.21 (AVSS), U18.24 (DVSS); no longer R11.2, R9.2
- net +5V_filt: now also C36.1, C38.1, C39.1, C40.1, C41.1, C42.1, U15.5 (~DIS), U15.6 (V+), U18.11 (DVDD), U18.13 (DVDD), U18.14 (AVDD), U18.15 (AVDD), U18.18 (AVDD)
- net +5V_sel: now also C33.1, U17.8 (V+)
- net f_ls_D10: now also J13.D27 (LA26_N)
- net f_ls_D8: now also J13.C27 (LA27_N)
- net f_ls_D9: now also J13.C26 (LA27_P)
- net f_ls_E0-DIR: now also J13.D26 (LA26_P)
- net f_ls_E0-EN: now also J13.G25 (LA22_N)
- net f_ls_E0-STEP: now also J13.G28 (LA25_N)
- net f_ls_E1-DIR: now also J13.G24 (LA22_P)
- net f_ls_E1-EN: now also J13.D23 (LA23_P)
- net f_ls_E1-STEP: now also J13.H26 (LA21_N)
- net f_ls_UART_RX: now also J13.H20 (LA15_N)
- net f_ls_UART_TX: now also J13.C19 (LA14_N)
- net f_ls_X-DIR: now also J13.H32 (LA28_N)
- net f_ls_X-EN: now also J13.G30 (LA29_P)
- net f_ls_X-MAX: now also J13.G15 (LA12_P)
- net f_ls_X-MIN: now also J13.H17 (LA11_N)
- net f_ls_X-STEP: now also J13.H31 (LA28_P)
- net f_ls_Y-DIR: now also J13.H28 (LA24_P)
- net f_ls_Y-EN: now also J13.G31 (LA29_N)
- net f_ls_Y-MAX: now also J13.D17 (LA13_P)
- net f_ls_Y-MIN: now also J13.G16 (LA12_N)
- net f_ls_Y-STEP: now also J13.D24 (LA23_N)
- net f_ls_Z-DIR: now also J13.G27 (LA25_P)
- net f_ls_Z-EN: now also J13.H34 (LA30_P)
- net f_ls_Z-MAX: now also J13.C18 (LA14_P)
- net f_ls_Z-MIN: now also J13.D18 (LA13_N)
- net f_ls_Z-STEP: now also J13.H29 (LA24_N)
- net fpga_SCL: now also J13.C30 (SCL)
- net fpga_SDA: now also J13.C31 (SDA)
- net ls_f_D10: now also J13.G10 (LA03_N)
- net ls_f_D8: now also J13.H11 (LA04_N)
- net ls_f_D9: now also J13.H10 (LA04_P)
- net ls_f_E0-DIR: now also J13.H16 (LA11_P)
- net ls_f_E0-EN: now also J13.H14 (LA07_N)
- net ls_f_E0-STEP: now also J13.C15 (LA10_N)
- net ls_f_E1-DIR: now also J13.H35 (LA30_N)
- net ls_f_E1-EN: now also J13.G12 (LA08_P)
- net ls_f_E1-STEP: now also J13.G33 (LA31_P)
- net ls_f_UART_RX: now also J13.H19 (LA15_P)
- net ls_f_UART_TX: now also J13.G18 (LA16_P)
- net ls_f_X-DIR: now also J13.D12 (LA05_N)
- net ls_f_X-EN: now also J13.C10 (LA06_P)
- net ls_f_X-MAX: now also J13.G36 (LA33_P)
- net ls_f_X-MIN: now also J13.G34 (LA31_N)
- net ls_f_X-STEP: now also J13.D11 (LA05_P)
- net ls_f_Y-DIR: now also J13.D14 (LA09_P)
- net ls_f_Y-EN: now also J13.C11 (LA06_N)
- net ls_f_Y-MAX: now also J13.G37 (LA33_N)
- net ls_f_Y-MIN: now also J13.H37 (LA32_P)
- net ls_f_Y-STEP: now also J13.G13 (LA08_N)
- net ls_f_Z-DIR: now also J13.C14 (LA10_P)
- net ls_f_Z-EN: now also J13.H13 (LA07_P)
- net ls_f_Z-MAX: now also J13.G19 (LA16_N)
- net ls_f_Z-MIN: now also J13.H38 (LA32_N)
- net ls_f_Z-STEP: now also J13.D15 (LA09_N)
- net r_THERM0: now also U17.3 (IN1+); no longer R8.1
- net r_THERM1: now also U17.5 (IN2+); no longer R10.1
- net at U14.12 (CLK): no longer J16.2 (Pin_2)
- net at J9.1 (In): now also C33.2
- net at J10.1 (In): now also C34.2
- net f_psc_ain renamed 5v_psc_ain
- net 5v_psc_ain: no longer U14.19 (VIN)
- net psc_d0 renamed 5V_psc_d0
- net psc_d1 renamed 5V_psc_d1
- net psc_d2 renamed 5V_psc_d2
- net psc_d3 renamed 5V_psc_d3
- net psc_d4 renamed 5V_psc_d4
- net psc_d5 renamed 5V_psc_d5
- net psc_d6 renamed 5V_psc_d6
- net psc_d7 renamed 5V_psc_d7
- new net: Q13.1 (C), U19.1 (CA1)
- new net: R45.2, U19.5 (E)
- new net: R40.2, R41.1, U15.4 (IN-)
- new net: R54.2, U19.14 (A)
- new net: Q16.1 (C), U19.8 (CA4)
- new net: R52.2, U19.13 (C)
- new net: R55.1, U19.7 (DP)
- new net: J13.J39 (VIO_B_M2C), J13.K40 (VIO_B_M2C)
- new net: Q15.1 (C), U19.6 (CA3)
- new net: R53.2, U19.16 (B)
- new net: J13.C35 (12P0V), J13.C37 (12P0V)
- new net: J13.C39 (3P3V), J13.D36 (3P3V), J13.D38 (3P3V), J13.D40 (3P3V)
- new net: J13.E39 (VADJ), J13.F40 (VADJ), J13.G39 (VADJ), J13.H40 (VADJ)
- new net: R44.2, U19.11 (F)
- new net: R43.2, U19.15 (G)
- new net: Q14.1 (C), U19.2 (CA2)
- new net: R51.2, U19.3 (D)
- new net: C35.2, R40.1
- new net 3V3_psc_ain: C37.1, R41.2, U15.1 (OUT), U18.19 (VIN)
- new net 3V3_psc_d0: U18.3 (D0)
- new net 3V3_psc_d1: U18.4 (D1)
- new net 3V3_psc_d2: U18.5 (D2)
- new net 3V3_psc_d3: U18.6 (D3)
- new net 3V3_psc_d4: U18.7 (D4)
- new net 3V3_psc_d5: U18.8 (D5)
- new net 3V3_psc_d6: U18.9 (D6)
- new net 3V3_psc_d7: U18.10 (D7)
- new net 3V3_psc_oe_n: U18.1 (~OE)
- new net 5V_psc_ain: U14.19 (VIN)
- new net 7seg_A1: Q13.2 (B)
- new net 7seg_A2: Q14.2 (B)
- new net 7seg_A3: Q15.2 (B)
- new net 7seg_A4: Q16.2 (B)
- new net 7seg_CA: R54.1
- new net 7seg_CB: R53.1
- new net 7seg_CC: R52.1
- new net 7seg_CD: R51.1
- new net 7seg_CE: R45.1
- new net 7seg_CF: R44.1
- new net 7seg_CG: R43.1
- new net 7seg_DP: R55.2
- new net f_dip_0: R56.2, SW1.1
- new net f_dip_1: R57.2, SW1.2
- new net f_dip_2: R58.2, SW1.3
- new net f_dip_3: R59.2, SW1.4
- new net f_dip_4: R60.2, SW1.5
- new net f_dip_5: R61.2, SW1.6
- new net f_dip_6: R62.2, SW1.7
- new net f_dip_7: R63.2, SW1.8
- new net hpc_n: J13.G9 (LA03_P), J3.1 (Pin_1), R42.2
- new net op_THERM0: R8.1, R9.2, U16.4 (AIN0)
- new net op_THERM1: R10.1, R11.2, U16.5 (AIN1)
- new net op_feedback0: R8.2, U17.1 (OUT1), U17.2 (IN1-)
- new net op_feedback1: R10.2, U17.6 (IN2-), U17.7 (OUT2)
- new net psc_clk: J16.2 (Pin_2), U18.12 (CLK)
- no-connect marks 13 -> 7
Other:
- note added: "CHECK THIS http://ww1.microchip.com/downloads/en/DeviceDoc/chapter%208.pdf"
- note added: "FMC Mezzanine Connector (HPC)"
- note added: "FMC low pin count and high pin count are compatible on a subset of pins. All RAMPS control signals are on the LPC GPIO. HPC_N jumper J3 to tell FPGA if HPC or LPC"
- note added: "HPC GPIO Pins"
- note added: "LPC GPIO Pins"
- note added: "Power & Shared Pins"
- note added: "REARRANGE FOR ROUTING"
- note added: "STEMMA QT connector"
- note added: "Shift to 5V Needs to be low latency"
- note added: "Single ended. Set up diff"
- note added: "To be added where needed during routing"
- note added: "UART Shifters"
- note added: "User Interface"
- note removed: "0-5V input become 0-3V3 Voltage divider (R2)/(R1+R2) = 1/3 = R2 = 5K, R1 = 10K"
- note removed: "ADD VOLTAGE FOLLOWERS?"
- note removed: "CHECK"
- note removed: "FMC Mezzanine Connector (LPC)"
- note removed: "UART Level Shifters"
- moved on the sheet: C1, C10, C11, C12, C13, C14, C15, C16, C17, C18, C19, C2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

Commit message: Cleanup. Needs review and then ready for routing.
Parts:
- removed J11, J12: Conn_Coaxial, symbol Connector:Conn_Coaxial
- removed R2, R34, R4, R5: 4.7k, Resistor_SMD:R_0805_2012Metric, symbol Device:R
- removed SW1: SW_DIP_x08, symbol Switch:SW_DIP_x08
- added J10: Conn_01x04_Socket, Connector_JST:JST_PH_B4B-PH-SM4-TB_1x04-1MP_P2.00mm_Vertical, symbol Connector:Conn_01x04_Socket
- added J16, J17: Conn_01x02_Pin, Connector_PinHeader_2.54mm:PinHeader_1x02_P2.54mm_Vertical, symbol Connector:Conn_01x02_Pin
- added R51, R56: 10K, Resistor_SMD:R_0805_2012Metric, symbol Device:R
- added R7: 4.7k, Resistor_SMD:R_0805_2012Metric, symbol Device:R
- added SW1: 219-8MST, SO16_219-8_CTS, symbol offramps_lib:219-8MST
- C11: renamed from C33; footprint (none) -> Capacitor_SMD:C_0805_2012Metric
- C12: renamed from C25; footprint (none) -> Capacitor_SMD:C_0805_2012Metric
- C13: renamed from C34; footprint (none) -> Capacitor_SMD:C_0805_2012Metric
- C14: renamed from C24; footprint (none) -> Capacitor_SMD:C_0805_2012Metric
- C15: renamed from C26; value C -> 100n; footprint (none) -> Capacitor_SMD:C_0805_2012Metric
- C16: renamed from C27; footprint (none) -> Capacitor_SMD:C_0805_2012Metric
- C17: renamed from C31; footprint (none) -> Capacitor_SMD:C_0805_2012Metric
- C18: renamed from C28; footprint (none) -> Capacitor_SMD:C_0805_2012Metric
- C19: renamed from C29; footprint (none) -> Capacitor_SMD:C_0805_2012Metric
- C20: renamed from C32; footprint (none) -> Capacitor_SMD:C_0805_2012Metric
- C22: renamed from C35; footprint (none) -> Capacitor_SMD:C_0805_2012Metric
- C25: renamed from C36; footprint (none) -> Capacitor_SMD:C_0805_2012Metric
- C26: renamed from C37; value C -> 100n; footprint (none) -> Capacitor_SMD:C_0805_2012Metric
- C27: renamed from C38; footprint (none) -> Capacitor_SMD:C_0805_2012Metric
- C28: renamed from C39; footprint (none) -> Capacitor_SMD:C_0805_2012Metric
- C29: renamed from C40; footprint (none) -> Capacitor_SMD:C_0805_2012Metric
- C30: renamed from C41; footprint (none) -> Capacitor_SMD:C_0805_2012Metric
- C31: renamed from C42; footprint (none) -> Capacitor_SMD:C_0805_2012Metric
- J4: renamed from J3; footprint (none) -> Connector_PinHeader_2.54mm:PinHeader_1x02_P2.54mm_Vertical
- J5: renamed from J9; footprint (none) -> Connector_Coaxial:SMA_Wurth_60312102114405_Vertical
- J7: renamed from J14; footprint (none) -> Connector_Coaxial:SMA_Wurth_60312102114405_Vertical
- J8: renamed from J10; footprint (none) -> Connector_Coaxial:SMA_Wurth_60312102114405_Vertical
- L1: footprint (none) -> Inductor_SMD:L_0805_2012Metric
- Q13, Q14, Q15, Q16: footprint (none) -> Package_TO_SOT_SMD:SOT-23
- R12: renamed from R3; footprint (none) -> Resistor_SMD:R_0805_2012Metric
- R13: renamed from R6; footprint (none) -> Resistor_SMD:R_0805_2012Metric
- R14: renamed from R12; footprint (none) -> Resistor_SMD:R_0805_2012Metric
- R15: renamed from R13; footprint (none) -> Resistor_SMD:R_0805_2012Metric
- R16: renamed from R14; footprint (none) -> Resistor_SMD:R_0805_2012Metric
- R17: renamed from R16; footprint (none) -> Resistor_SMD:R_0805_2012Metric
- R18: footprint (none) -> Resistor_SMD:R_0805_2012Metric
- R19: renamed from R28; footprint (none) -> Resistor_SMD:R_0805_2012Metric
- R2: renamed from R21; footprint (none) -> Resistor_SMD:R_0805_2012Metric
- R20: renamed from R15; footprint (none) -> Resistor_SMD:R_0805_2012Metric
- R21: renamed from R17; footprint (none) -> Resistor_SMD:R_0805_2012Metric
- R22: renamed from R27; footprint (none) -> Resistor_SMD:R_0805_2012Metric
- R23: renamed from R29; footprint (none) -> Resistor_SMD:R_0805_2012Metric
- R24: renamed from R42; footprint (none) -> Resistor_SMD:R_0805_2012Metric
- R25: renamed from R30; footprint (none) -> Resistor_SMD:R_0805_2012Metric
- R26: renamed from R50; footprint (none) -> Resistor_SMD:R_0805_2012Metric
- R27: renamed from R31; footprint (none) -> Resistor_SMD:R_0805_2012Metric
- R3: renamed from R24; footprint (none) -> Resistor_SMD:R_0805_2012Metric
- R30: renamed from R40; footprint (none) -> Resistor_SMD:R_0805_2012Metric
- R31: renamed from R41; footprint (none) -> Resistor_SMD:R_0805_2012Metric
- R32: renamed from R33; now not fitted
- R33: renamed from R37; now not fitted
- R34: renamed from R56; footprint (none) -> Resistor_SMD:R_0805_2012Metric
- R35: renamed from R53; footprint (none) -> Resistor_SMD:R_0805_2012Metric
- R36: renamed from R51; footprint (none) -> Resistor_SMD:R_0805_2012Metric
- R37: renamed from R44; footprint (none) -> Resistor_SMD:R_0805_2012Metric
- R38: renamed from R55; footprint (none) -> Resistor_SMD:R_0805_2012Metric
- R39: renamed from R8; footprint (none) -> Resistor_SMD:R_0805_2012Metric
- R40: renamed from R9; footprint (none) -> Resistor_SMD:R_0805_2012Metric
- R41: renamed from R57; footprint (none) -> Resistor_SMD:R_0805_2012Metric
- R42: renamed from R52; footprint (none) -> Resistor_SMD:R_0805_2012Metric
- R43: renamed from R45; footprint (none) -> Resistor_SMD:R_0805_2012Metric
- R44: renamed from R43; footprint (none) -> Resistor_SMD:R_0805_2012Metric
- R45: renamed from R58; footprint (none) -> Resistor_SMD:R_0805_2012Metric
- R46: renamed from R54; footprint (none) -> Resistor_SMD:R_0805_2012Metric
- R47: renamed from R10; footprint (none) -> Resistor_SMD:R_0805_2012Metric
- R48: renamed from R11; footprint (none) -> Resistor_SMD:R_0805_2012Metric
- R49: renamed from R59; footprint (none) -> Resistor_SMD:R_0805_2012Metric
- R5: renamed from R22; footprint (none) -> Resistor_SMD:R_0805_2012Metric
- R50: renamed from R38; now not fitted
- R52: renamed from R35; now not fitted
- R53: renamed from R60; footprint (none) -> Resistor_SMD:R_0805_2012Metric
- R54: renamed from R61; footprint (none) -> Resistor_SMD:R_0805_2012Metric
- R55: renamed from R39; now not fitted
- R57: renamed from R36; now not fitted
- R58: renamed from R62; footprint (none) -> Resistor_SMD:R_0805_2012Metric
- R59: renamed from R63; footprint (none) -> Resistor_SMD:R_0805_2012Metric
- R6: renamed from R25; footprint (none) -> Resistor_SMD:R_0805_2012Metric
- R60: renamed from R46; footprint (none) -> Resistor_SMD:R_0805_2012Metric
- R61: renamed from R19; footprint (none) -> Resistor_SMD:R_0805_2012Metric
- R62: renamed from R47; footprint (none) -> Resistor_SMD:R_0805_2012Metric
- R63: renamed from R48; footprint (none) -> Resistor_SMD:R_0805_2012Metric
- R64: renamed from R20; footprint (none) -> Resistor_SMD:R_0805_2012Metric
- R65: renamed from R49; footprint (none) -> Resistor_SMD:R_0805_2012Metric
- R8: renamed from R23; footprint (none) -> Resistor_SMD:R_0805_2012Metric
- R9: renamed from R26; footprint (none) -> Resistor_SMD:R_0805_2012Metric
- TP1: renamed from TP?; footprint (none) -> TestPoint:TestPoint_Loop_D2.50mm_Drill1.0mm
- TP2: renamed from TP1; footprint (none) -> TestPoint:TestPoint_Loop_D2.50mm_Drill1.0mm
- TP3: renamed from TP2; footprint (none) -> TestPoint:TestPoint_Loop_D2.50mm_Drill1.0mm
- TP4: renamed from TP3; footprint (none) -> TestPoint:TestPoint_Loop_D2.50mm_Drill1.0mm
- TP5: renamed from TP4; footprint (none) -> TestPoint:TestPoint_Loop_D2.50mm_Drill1.0mm
- TP6: renamed from TP5; footprint (none) -> TestPoint:TestPoint_Loop_D2.50mm_Drill1.0mm
- U11: renamed from U15; footprint MK06A -> offramps_lib:MK06A
- U12: renamed from U18; footprint MTC24 -> offramps_lib:MTC24_TEX
- U14: renamed from U17; footprint VSSOP8_DGK_TEX -> offramps_lib:VSSOP8_DGK_TEX
- U6: renamed from U12; footprint MK06A -> offramps_lib:MK06A
- U7: renamed from U14; footprint MTC24_TEX -> offramps_lib:MTC24_TEX
- renumbered C7 to C1, C6 to C10, C9 to C2, C17 to C21, C15 to C23, C16 to C24, C8 to C3, C19 to C32, C18 to C33, C20 to C34, C21 to C35, C13 to C36, C22 to C37, C14 to C38, C23 to C39, C11 to C4, C30 to C40, C1 to C41, C2 to C42, C10 to C5, C12 to C6, C3 to C7, C4 to C8, C5 to C9, J5 to J11, J4 to J12, J15 to J13, J6 to J14, J7 to J15, J13 to J3, J16 to J6, J8 to J9, Q5 to Q1, Q4 to Q10, Q8 to Q2, Q6 to Q3, Q9 to Q4, Q7 to Q5, Q10 to Q6, Q1 to Q7, Q2 to Q8, Q3 to Q9, R32 to R28, R7 to R29, U5 to U1, U8 to U10, U9 to U13, U16 to U15, U11 to U16, U7 to U17, U19 to U18, U1 to U19, U4 to U3, U6 to U4, U3 to U5, U13 to U8, U10 to U9
Connections:
- net +3V3_sel: now also J10.3 (Pin_3), J10.4 (Pin_4), J16.1 (Pin_1), J17.1 (Pin_1), R51.1, R56.1, R7.2, SW1.10, SW1.11, SW1.12, SW1.13, SW1.14, SW1.15, SW1.16, SW1.9; no longer R1.1, U1.10 (OE), U2.10 (OE), U3.10 (OE), U4.10 (OE), U5.10 (OE)
- net f_dip_0: now also SW1.1
- net f_dip_1: now also SW1.2
- net f_dip_2: now also SW1.3
- net f_dip_3: now also SW1.4
- net f_dip_4: now also SW1.5
- net f_dip_5: now also SW1.6
- net f_dip_6: now also SW1.7
- net f_dip_7: now also SW1.8
- net fpga_SCL: now also J10.1 (Pin_1), R51.2
- net fpga_SDA: now also J10.2 (Pin_2), R56.2
- net ext_scope_clk renamed ext_psc_clk
- net f_scope_clk renamed fpga_psc_clk
- new net 3V3_5V_tristate: J16.2 (Pin_2), R7.1, U2.10 (OE), U5.10 (OE)
- new net 5V_3V3_tristate: J17.2 (Pin_2), R1.1, U1.10 (OE), U3.10 (OE), U4.10 (OE)
Other:
- note added: "Stemma QT compatible JST"
- note added: "Swap for 10 resistor chip"
- note added: "https://github.com/newaetech/chipwhisperer/tree/develop/hardware/capture/chipwhisperer-nano"
- note removed: "STEMMA QT connector"
- note removed: "Single ended. Set up diff"
- moved on the sheet: C1, C11, C13, C2, C3, C37, C39, C4, C5, C6, J14, J4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

Commit message: Updated symbols to match offramps_lib footprints
Parts:
- J1, J2: footprint jblocklove_kicad:arduino_mega_shield -> offramps_lib:arduino_mega_shield
- J11, J15: footprint kiwih_kicad:WR-TBL-TermBlock-2Pos-90Deg-5.08mm -> offramps_lib:WR-TBL-TermBlock-2Pos-90Deg-5.08mm
- J12: footprint jblocklove_kicad:3-way_jumper -> offramps_lib:3-way_jumper
- SW1: footprint SO16_219-8_CTS -> offramps_lib:WR-TBL-TermBlock-2Pos-90Deg-5.08mm
- U1, U2, U3, U4, U5, U8: footprint external_footprints:SOP65P640X120-20N -> offramps_lib:SOP65P640X120-20N
Changed lines of the file:
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@@
 			)
 		)
-		(property "Footprint" "external_footprints:SOP65P640X120-20N"
+		(property "Footprint" "offramps_lib:SOP65P640X120-20N"
 			(at 63.5 215.9 0)
 			(effects
@@
 			)
 		)
-		(property "Footprint" "jblocklove_kicad:arduino_mega_shield"
+		(property "Footprint" "offramps_lib:arduino_mega_shield"
 			(at 40.64 116.84 90)
 			(effects
@@
 			)
 		)
-		(property "Footprint" "jblocklove_kicad:arduino_mega_shield"
+		(property "Footprint" "offramps_lib:arduino_mega_shield"
 			(at 40.64 63.5 90)
 			(effects
@@
 			)
 		)
-		(property "Footprint" "jblocklove_kicad:arduino_mega_shield"
+		(property "Footprint" "offramps_lib:arduino_mega_shield"
 			(at 40.64 91.44 90)
 			(effects
@@
 			)
 		)
-		(property "Footprint" "jblocklove_kicad:arduino_mega_shield"
+		(property "Footprint" "offramps_lib:arduino_mega_shield"
 			(at 153.67 60.96 90)
 			(effects
@@
 			)
 		)
-		(property "Footprint" "jblocklove_kicad:arduino_mega_shield"
+		(property "Footprint" "offramps_lib:arduino_mega_shield"
 			(at 128.27 55.88 90)
 			(effects
@@
 			)
 		)
-		(property "Footprint" "jblocklove_kicad:arduino_mega_shield"
+		(property "Footprint" "offramps_lib:arduino_mega_shield"
 			(at 64.77 116.84 90)
 			(effects
@@
 			)
 		)
-		(property "Footprint" "kiwih_kicad:WR-TBL-TermBlock-2Pos-90Deg-5.08mm"
+		(property "Footprint" "offramps_lib:WR-TBL-TermBlock-2Pos-90Deg-5.08mm"
 			(at 626.11 83.82 0)
 			(effects
@@
 			)
 		)
-		(property "Footprint" "external_footprints:SOP65P640X120-20N"
+		(property "Footprint" "offramps_lib:SOP65P640X120-20N"
 			(at 358.14 279.4 0)
 			(effects
@@
 			)
 		)
-		(property "Footprint" "external_footprints:SOP65P640X120-20N"
+		(property "Footprint" "offramps_lib:SOP65P640X120-20N"
 			(at 144.78 213.36 0)
 			(effects
@@
 			)
 		)
-		(property "Footprint" "external_footprints:SOP65P640X120-20N"
+		(property "Footprint" "offramps_lib:SOP65P640X120-20N"
 			(at 359.41 226.06 0)
 			(effects
@@
 			)
 		)
-		(property "Footprint" "kiwih_kicad:WR-TBL-TermBlock-2Pos-90Deg-5.08mm"
+		(property "Footprint" "offramps_lib:WR-TBL-TermBlock-2Pos-90Deg-5.08mm"
 			(at 668.02 57.15 0)
 			(effects
@@
 			)
 		)
-		(property "Footprint" "jblocklove_kicad:arduino_mega_shield"
+		(property "Footprint" "offramps_lib:arduino_mega_shield"
 			(at 153.67 114.3 90)
 			(effects
@@
 			)
 		)
-		(property "Footprint" "external_footprints:SOP65P640X120-20N"
+		(property "Footprint" "offramps_lib:SOP65P640X120-20N"
 			(at 295.91 231.14 0)
 			(effects
@@
 			)
 		)
-		(property "Footprint" "jblocklove_kicad:arduino_mega_shield"
+		(property "Footprint" "offramps_lib:arduino_mega_shield"
 			(at 66.04 91.44 90)
 			(effects
@@
 			)
 		)
-		(property "Footprint" "jblocklove_kicad:3-way_jumper"
+		(property "Footprint" "offramps_lib:3-way_jumper"
 			(at 627.38 43.18 0)
 			(effects
@@
 			)
 		)
-		(property "Footprint" "jblocklove_kicad:arduino_mega_shield"
+		(property "Footprint" "offramps_lib:arduino_mega_shield"
 			(at 66.04 58.42 90)
 			(effects
@@
 			)
 		)
-		(property "Footprint" "external_footprints:SOP65P640X120-20N"
+		(property "Footprint" "offramps_lib:SOP65P640X120-20N"
 			(at 384.81 355.6 0)
 			(effects
@@
 			)
 		)
-		(property "Footprint" "jblocklove_kicad:arduino_mega_shield"
+		(property "Footprint" "offramps_lib:arduino_mega_shield"
 			(at 129.54 114.3 90)
 			(effects
@@
 			)
 		)
-		(property "Footprint" "jblocklove_kicad:arduino_mega_shield"
+		(property "Footprint" "offramps_lib:arduino_mega_shield"
 			(at 24.13 135.89 90)
 			(effects
@@
 			)
 		)
-		(property "Footprint" "jblocklove_kicad:arduino_mega_shield"
+		(property "Footprint" "offramps_lib:arduino_mega_shield"
 			(at 171.45 134.62 90)
 			(effects
@@
 			)
 		)
-		(property "Footprint" "jblocklove_kicad:arduino_mega_shield"
+		(property "Footprint" "offramps_lib:arduino_mega_shield"
 			(at 128.27 88.9 90)
 			(effects
@@
 			)
 		)
-		(property "Footprint" "SO16_219-8_CTS"
+		(property "Footprint" "offramps_lib:WR-TBL-TermBlock-2Pos-90Deg-5.08mm"
 			(at 613.41 346.71 0)
 			(effects
@@
 			)
 		)
-		(property "Footprint" "jblocklove_kicad:arduino_mega_shield"
+		(property "Footprint" "offramps_lib:arduino_mega_shield"
 			(at 153.67 88.9 90)
 			(effects

Commit message: Review'd and added notes to schematic
Parts:
- added Q17, Q18: BSS138, Package_TO_SOT_SMD:SOT-23, symbol Transistor_FET:BSS138
- added R10, R4: 10k, Resistor_SMD:R_0805_2012Metric, symbol Device:R
- J5, J7, J8: footprint Connector_Coaxial:SMA_Wurth_60312102114405_Vertical -> Connector_Coaxial:MMCX_Molex_73415-1471_Vertical
- U14: footprint offramps_lib:VSSOP8_DGK_TEX -> VSSOP8_DGK_TEX
Connections:
- net ls_f_X-MIN is gone; now on net +3V3_sel: J3.G34 (LA31_N), Q1.3 (D), R2.1
- net +3V3_sel: now also Q18.3 (D), R10.2, R4.2
- net +5V_sel: now also Q17.3 (D)
- net fpga_SCL: now also R33.2; no longer R32.2
- net fpga_SDA: now also R32.2; no longer R33.2
- net op_feedback0: now also U14.6 (IN2-), U14.7 (OUT2); no longer U14.1 (OUT1), U14.2 (IN1-)
- net op_feedback1: now also U14.1 (OUT1), U14.2 (IN1-); no longer U14.6 (IN2-), U14.7 (OUT2)
- net r_THERM0: now also U14.5 (IN2+); no longer U14.3 (IN1+)
- net r_THERM1: now also U14.3 (IN1+); no longer U14.5 (IN2+)
- net r_X-MIN: now also Q18.1 (G)
- new net: Q17.2 (S), R10.1
- new net: Q18.2 (S), R4.1
Other:
- note added: "***"
- note added: "0V"
- note added: "3V3"
- note added: "3V3 input clock"
- note added: "5V"
- note added: "5V0 output clock"
- note added: "< Switch depress"
- note added: "< Switch press"
- note added: "Double check that the FET is oriented properly (Drain and source are not switched) and that TX/RX directionality doesn't matter for FET direction"
- note added: "I Changed the footprint for this coaxial connector to the one with 5 posts. We should look at the dimensions with the one we are planning on using during part sourcing to make sure it will work."
- note added: "I couldn't find any 10K arrays on JLC PCB. Maybe we can source one of Digikey, but it will be more expensive than 10 discrete resistors (both on Digikey and JLC) Leaving this as is for now."
- note added: "I modified this symbol"
- note added: "I think these NFETs are wired incorrectly. The 3v3 is connected to the source (which I think should always be connected top GND) If this is the expected behavior on the switches, I think a circuit like this should work for each of the end stops:"
- note added: "I2C Pull ups are usually 4.7K"
- note added: "Notes: Some of the schematics are hard to understand. (might lead to more errors) - I suggest using less connected labels and connect wires / resistors directly to components - Some signals are ambiguous in terms of voltage (when labels are used) Should fix convention for low enable pins (nEN vs ~EN vs *EN) There are many unconnected pins - some are intentional, which should be denoted with an un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"
- note added: "This type of circuit should work for the clock translation (at low speed)"
- note added: "This will draw 0.5mA A lower resistance --> Higher current --> Faster switching --> Better slew Can lower resistance in future depending on required speed"
- moved on the sheet: C37, C39, Q8, R13, R15, R32, R33, R39, R40, R47, R48, U15
