File: kicad/offramps/offramps.kicad_sch (KiCad schematic)
At the start: 195 parts, among them J10 Conn_01x04_Socket, J11 Screw_Terminal_01x02, J12 Conn_01x04_Pin, J13 Micro_SD_Card, J14 Conn_01x03_Male, J15 Screw_Terminal_01x02, J16 Conn_01x02_Pin, J17 Conn_01x02_Pin, J3 VITA_57.1_FMC_HPC_Carrier, J4 Conn_01x02_Pin, J5 Conn_Coaxial, J6 Conn_01x03_Male, J7 Conn_Coaxial, J8 Conn_Coaxial, J9 Conn_01x06_Male, Q1 BSS138, Q10 BSS138, Q11 BSS138, Q12 BSS138, Q13 NPN, Q14 NPN, Q15 NPN, Q16 NPN, Q17 BSS138, Q18 BSS138, Q2 BSS138, Q3 BSS138, Q4 BSS138, Q5 BSS138, Q6 BSS138, Q7 BSS138, Q8 BSS138, Q9 BSS138, SW1 219-8MST, U1 TXB0108PWR, U10 MCP4725xxx-xCH, U11 LMH6611MK/NOPB, U12 ADC1173CIMTC/NOPB, U13 MCP4725xxx-xCH, U14 POPA2994IDGKR, U15 ADS1114IDGS, U16 LIS2MDLTR, U17 LSM6DSRTR, U18 LTC-4627JR, U19 AMS1117-3.3, U2 TXB0108PWR, U3 TXB0108PWR, U4 TXB0108PWR, U5 TXB0108PWR, U6 LMH6611MK/NOPB, U7 ADC1175CIMTC/NOPB, U8 TXB0108PWR, U9 PTMUX4053PWR

Commit message: Schematic updates
Parts:
- removed Q18: BSS138, Package_TO_SOT_SMD:SOT-23, symbol Transistor_FET:BSS138
- removed R4: 10k, Resistor_SMD:R_0805_2012Metric, symbol Device:R
- added JP26, JP27: Jumper_3_Open, Connector_PinHeader_2.54mm:PinHeader_1x03_P2.54mm_Vertical, symbol Jumper:Jumper_3_Open
- added L2: 10u, Inductor_SMD:L_0805_2012Metric, symbol Device:L
- added Q25, Q26, Q27, Q28, Q29, Q30: BSS138, Package_TO_SOT_SMD:SOT-23, symbol Transistor_FET:BSS138
- added R11: 10R, Resistor_SMD:R_0805_2012Metric, symbol Device:R
- added R72, R73, R74, R75, R76, R77: 10k, Resistor_SMD:R_0805_2012Metric, symbol Device:R
Connections:
- net ls_f_X-MAX is gone; now on net +3V3_sel: J3.G36 (LA33_P), Q2.3 (D), R3.1
- net ls_f_Y-MAX is gone; now on net +3V3_sel: J3.G37 (LA33_N), Q4.3 (D), R6.1
- net ls_f_Y-MIN is gone; now on net +3V3_sel: J3.H37 (LA32_P), Q3.3 (D), R5.1
- net ls_f_Z-MAX is gone; now on net +3V3_sel: J3.G19 (LA16_N), Q6.3 (D), R9.1
- net ls_f_Z-MIN is gone; now on net +3V3_sel: J3.H38 (LA32_N), Q5.3 (D), R8.1
- net +3V3_sel: now also J3.C39 (3P3V), J3.D36 (3P3V), J3.D38 (3P3V), J3.D40 (3P3V), L2.1, Q25.3 (D), Q26.3 (D), Q27.3 (D), Q28.3 (D), Q29.3 (D), Q30.3 (D), R72.2, R73.2, R74.2, R75.2, R76.2, R77.2; no longer C22.1
- net 3V3_psc_d0: now also J3.F13 (HA12_P)
- net 3V3_psc_d1: now also J3.F14 (HA12_N)
- net 3V3_psc_d2: now also J3.E12 (HA13_P)
- net 3V3_psc_d3: now also J3.E13 (HA13_N)
- net 3V3_psc_d4: now also J3.J15 (HA14_P)
- net 3V3_psc_d5: now also J3.J16 (HA14_N)
- net 3V3_psc_d6: now also J3.F16 (HA15_P)
- net 3V3_psc_d7: now also J3.F17 (HA15_N)
- net 5V_psc_d0: now also J3.E7 (HA05_N)
- net 5V_psc_d1: now also J3.K10 (HA06_P)
- net 5V_psc_d2: now also J3.K11 (HA06_N)
- net 5V_psc_d3: now also J3.J9 (HA07_P)
- net 5V_psc_d4: now also J3.J10 (HA07_N)
- net 5V_psc_d5: now also J3.F10 (HA08_P)
- net 5V_psc_d6: now also J3.F11 (HA08_N)
- net 5V_psc_d7: now also J3.E9 (HA09_P)
- net 5V_psc_oe_n: now also U7.1 (~OE)
- net 7seg_CA: now also J3.K23 (HA23_N)
- net 7seg_CB: now also J3.K22 (HA23_P)
- net 7seg_CC: now also J3.J22 (HA22_N)
- net 7seg_CD: now also J3.J21 (HA22_P)
- net 7seg_CE: now also J3.K20 (HA21_N)
- net 7seg_CF: now also J3.K19 (HA21_P)
- net 7seg_CG: now also J3.E19 (HA20_N)
- net 7seg_DP: now also J3.E18 (HA20_P)
- net f_dip_0: now also J3.F20 (HA19_N)
- net f_dip_1: now also J3.F19 (HA19_P)
- net f_dip_2: now also J3.J19 (HA18_N)
- net f_dip_3: now also J3.J18 (HA18_P)
- net f_dip_4: now also J3.K17 (HA17_N_CC)
- net f_dip_5: now also J3.K16 (HA17_P_CC)
- net f_dip_6: now also J3.E16 (HA16_N)
- net f_dip_7: now also J3.E15 (HA16_P)
- net f_sd_clk: now also J3.D8 (LA01_P_CC)
- net f_sd_cmd: now also J3.E10 (HA09_N)
- net f_sd_dat0: now also J3.K14 (HA10_N)
- net f_sd_dat1: now also J3.K13 (HA10_P)
- net f_sd_dat2: now also J3.J13 (HA11_N)
- net f_sd_dat3: now also J3.J12 (HA11_P)
- net fpga_psc_clk: now also J3.G6 (LA00_P_CC)
- net psc_clk: now also Q17.1 (G)
- net r_SCL: now also JP26.1 (A)
- net r_SDA: now also JP27.1 (A)
- net r_X-MAX: now also Q29.1 (G)
- net r_X-MIN: now also Q30.1 (G)
- net r_Y-MAX: now also Q28.1 (G)
- net r_Y-MIN: now also Q27.1 (G)
- net r_Z-MAX: now also Q26.1 (G)
- net r_Z-MIN: now also Q25.1 (G)
- net u_SCL: now also JP26.2 (C)
- net u_SDA: now also JP27.2 (C)
- net psc_clk_5V: now reaches Q17.2 (S), R10.1
- net psc_clk_5V: now also U7.12 (CLK)
- new net: Q27.2 (S), R74.1
- new net: Q26.2 (S), R73.1
- new net: Q28.2 (S), R75.1
- new net: Q25.2 (S), R72.1
- new net: L2.2, R11.2
- new net: Q29.2 (S), R76.1
- new net: Q30.2 (S), R77.1
- new net +3V3_filt: C22.1, R11.1
- no-connect marks 7 -> 9
Other:
- note added: "I2C EXT"
- note added: "Orignal Design: (Excluded from board)"
- note removed: "***"
- note removed: "0V"
- note removed: "3V3"
- note removed: "5V"
- note removed: "< Switch depress"
- note removed: "< Switch press"
- note removed: "Double check that the FET is oriented properly (Drain and source are not switched) and that TX/RX directionality doesn't matter for FET direction"
- note removed: "I Changed the footprint for this coaxial connector to the one with 5 posts. We should look at the dimensions with the one we are planning on using during part sourcing to make sure it will work."
- note removed: "I couldn't find any 10K arrays on JLC PCB. Maybe we can source one of Digikey, but it will be more expensive than 10 discrete resistors (both on Digikey and JLC) Leaving this as is for now."
- note removed: "I modified this symbol"
- note removed: "I think these NFETs are wired incorrectly. The 3v3 is connected to the source (which I think should always be connected top GND) If this is the expected behavior on the switches, I think a circuit like this should work for each of the end stops:"
- note removed: "I2C Pull ups are usually 4.7K"
- note removed: "Notes: Some of the schematics are hard to understand. (might lead to more errors) - I suggest using less connected labels and connect wires / resistors directly to components - Some signals are ambiguous in terms of voltage (when labels are used) Should fix convention for low enable pins (nEN vs ~EN vs *EN) There are many unconnected pins - some are intentional, which should be denoted with an un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"
- moved on the sheet: J3C, J3D, L1, Q1, Q17, Q2, Q3, Q4, Q5, Q6, R10, R2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

Commit message: Updates
Parts:
- SW1: footprint offramps_lib:WR-TBL-TermBlock-2Pos-90Deg-5.08mm -> offramps_lib:SO16_219-8_CTS
Other:
- note added: "HPC is missing pin B40"
Changed lines of the file:
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@@
 		)
 	)
+	(polyline
+		(pts
+			(xy 311.15 -27.94) (xy 328.93 -27.94)
+		)
+		(stroke
+			(width 0)
+			(type default)
+		)
+	)
 	(wire
 		(pts
@@
 		)
 	)
+	(polyline
+		(pts
+			(xy 311.15 54.61) (xy 311.15 -27.94)
+		)
+		(stroke
+			(width 0)
+			(type default)
+		)
+	)
 	(wire
 		(pts
@@
 		)
 	)
+	(text "HPC is missing pin B40"
+		(exclude_from_sim no)
+		(at 319.024 -30.988 0)
+		(effects
+			(font
+				(size 1.27 1.27)
+			)
+		)
+	)
 	(text "Power analysis clock selection"
 		(exclude_from_sim no)
@@
 		(pin "6"
 		)
-		(pin "6"
+		(pin "7"
 		)
 		(pin "8"
@@
 			)
 		)
-		(property "Footprint" "offramps_lib:WR-TBL-TermBlock-2Pos-90Deg-5.08mm"
+		(property "Footprint" "offramps_lib:SO16_219-8_CTS"
 			(at 613.41 346.71 0)
 			(effects

Commit message: small updates + fixes
Parts:
- U14: footprint VSSOP8_DGK_TEX -> offramps_lib:VSSOP8_DGK_TEX
Connections:
- net +3V3_sel: no longer C1.2, C10.2, C14.2, C15.2, C16.2, C17.2, C18.2, C19.2, C2.2, C20.2, C21.2, C23.2, C24.2, C25.2, C26.2, C27.2, C28.2, C29.2, C3.2, C30.2, C31.2, C32.2, C33.2, C34.2, C35.2, C36.2, C37.1, C38.2, C39.1, C4.2, C40.2, C41.2, C42.2, C5.2, C6.2, C7.2, C8.2, C9.2, D1.1 (K), D2.1 (K), J1.25 (GND), J1.26 (GND), J1.6 (GND), J1.7 (GND), J1.83 (GND), J10.4 (Pin_4), J11.2 (Pin_2), J13.6 (VSS), J13.9 (SHIELD), J15.2 (Pin_2), J2.25 (GND), J2.26 (GND), J2.6 (GND), J2.7 (GND), J2.83 (GND), J3.A1 (GND), J3.A12 (GND), J3.A13 (GND), J3.A16 (GND), J3.A17 (GND), J3.A20 (GND), J3.A21 (GND), J3.A24 (GND), J3.A25 (GND), J3.A28 (GND), J3.A29 (GND), J3.A32 (GND), J3.A33 (GND), J3.A36 (GND), J3.A37 (GND), J3.A4 (GND), J3.A40 (GND), J3.A5 (GND), J3.A8 (GND), J3.A9 (GND), J3.B10 (GND), J3.B11 (GND), J3.B14 (GND), J3.B15 (GND), J3.B18 (GND), J3.B19 (GND), J3.B2 (GND), J3.B22 (GND), J3.B23 (GND), J3.B26 (GND), J3.B27 (GND), J3.B3 (GND), J3.B30 (GND), J3.B31 (GND), J3.B34 (GND), J3.B35 (GND), J3.B38 (GND), J3.B39 (GND), J3.B6 (GND), J3.B7 (GND), J3.C1 (GND), J3.C12 (GND), J3.C13 (GND), J3.C16 (GND), J3.C17 (GND), J3.C20 (GND), J3.C21 (GND), J3.C24 (GND), J3.C25 (GND), J3.C28 (GND), J3.C29 (GND), J3.C32 (GND), J3.C33 (GND), J3.C36 (GND), J3.C38 (GND), J3.C4 (GND), J3.C40 (GND), J3.C5 (GND), J3.C8 (GND), J3.C9 (GND), J3.D10 (GND), J3.D13 (GND), J3.D16 (GND), J3.D19 (GND), J3.D2 (GND), J3.D22 (GND), J3.D25 (GND), J3.D28 (GND), J3.D3 (GND), J3.D37 (GND), J3.D39 (GND), J3.D6 (GND), J3.D7 (GND), J3.E1 (GND), J3.E11 (GND), J3.E14 (GND), J3.E17 (GND), J3.E20 (GND), J3.E23 (GND), J3.E26 (GND), J3.E29 (GND), J3.E32 (GND), J3.E35 (GND), J3.E38 (GND), J3.E4 (GND), J3.E40 (GND), J3.E5 (GND), J3.E8 (GND), J3.F12 (GND), J3.F15 (GND), J3.F18 (GND), J3.F2 (GND), J3.F21 (GND), J3.F24 (GND), J3.F27 (GND), J3.F3 (GND), J3.F30 (GND), J3.F33 (GND), J3.F36 (GND), J3.F39 (GND), J3.F6 (GND), J3.F9 (GND), J3.G1 (GND), J3.G11 (GND), J3.G14 (GND), J3.G17 (GND), J3.G20 (GND), J3.G23 (GND), J3.G26 (GND), J3.G29 (GND), J3.G32 (GND), J3.G35 (GND), J3.G38 (GND), J3.G4 (GND), J3.G40 (GND), J3.G5 (GND), J3.G8 (GND), J3.H12 (GND), J3.H15 (GND), J3.H18 (GND), J3.H21 (GND), J3.H24 (GND), J3.H27 (GND), J3.H3 (GND), J3.H30 (GND), J3.H33 (GND), J3.H36 (GND), J3.H39 (GND), J3.H6 (GND), J3.H9 (GND), J3.J1 (GND), J3.J11 (GND), J3.J14 (GND), J3.J17 (GND), J3.J20 (GND), J3.J23 (GND), J3.J26 (GND), J3.J29 (GND), J3.J32 (GND), J3.J35 (GND), J3.J38 (GND), J3.J4 (GND), J3.J40 (GND), J3.J5 (GND), J3.J8 (GND), J3.K12 (GND), J3.K15 (GND), J3.K18 (GND), J3.K2 (GND), J3.K21 (GND), J3.K24 (GND), J3.K27 (GND), J3.K3 (GND), J3.K30 (GND), J3.K33 (GND), J3.K36 (GND), J3.K39 (GND), J3.K6 (GND), J3.K9 (GND), J4.2 (Pin_2), J5.2 (Ext), J7.2 (Ext), J8.2 (Ext), J9.6 (Pin_6), R1.2, R10.2, R2.2, R28.1, R29.2, R3.2, R40.1, R48.1, R5.2, R6.2, R7.2, R72.2, R73.2, R74.2, R75.2, R76.2, R77.2, R8.2, R9.2, SW1.10, SW1.11, SW1.12, SW1.13, SW1.14, SW1.15, SW1.16, SW1.9, TP2.1, TP3.1, TP4.1, TP5.1, TP6.1, U1.11 (GND), U10.2 (VSS), U11.2 (V-), U11.3 (IN+), U12.2 (DVSS), U12.20 (AVSS), U12.21 (AVSS), U12.24 (DVSS), U13.2 (VSS), U13.6 (A0), U14.4 (V-), U15.3 (GND), U16.6 (GND), U16.8 (GND), U17.6 (GND), U17.7 (GND), U19.1 (GND), U2.11 (GND), U3.11 (GND), U4.11 (GND), U5.11 (GND), U6.2 (V-), U6.3 (IN+), U7.2 (DVSS), U7.20 (AVSS), U7.21 (AVSS), U7.24 (DVSS), U8.11 (GND), U9.6 (*EN), U9.7 (VSS), U9.8 (GND)
- new net GND: C1.2, C10.2, C14.2, C15.2, C16.2, C17.2, C18.2, C19.2, C2.2, C20.2, C21.2, C23.2, C24.2, C25.2, C26.2, C27.2, C28.2, C29.2, C3.2, C30.2, C31.2, C32.2, C33.2, C34.2, C35.2, C36.2, C37.1, C38.2, C39.1, C4.2, C40.2, C41.2, C42.2, C5.2, C6.2, C7.2, C8.2, C9.2, D1.1 (K), D2.1 (K), J1.25 (GND), J1.26 (GND), J1.6 (GND), J1.7 (GND), J1.83 (GND), J10.4 (Pin_4), J11.2 (Pin_2), J13.6 (VSS), J13.9 (SHIELD), J15.2 (Pin_2), J2.25 (GND), J2.26 (GND), J2.6 (GND), J2.7 (GND), J2.83 (GND), J3.A1 (GND), J3.A12 (GND), J3.A13 (GND), J3.A16 (GND), J3.A17 (GND), J3.A20 (GND), J3.A21 (GND), J3.A24 (GND), J3.A25 (GND), J3.A28 (GND), J3.A29 (GND), J3.A32 (GND), J3.A33 (GND), J3.A36 (GND), J3.A37 (GND), J3.A4 (GND), J3.A40 (GND), J3.A5 (GND), J3.A8 (GND), J3.A9 (GND), J3.B10 (GND), J3.B11 (GND), J3.B14 (GND), J3.B15 (GND), J3.B18 (GND), J3.B19 (GND), J3.B2 (GND), J3.B22 (GND), J3.B23 (GND), J3.B26 (GND), J3.B27 (GND), J3.B3 (GND), J3.B30 (GND), J3.B31 (GND), J3.B34 (GND), J3.B35 (GND), J3.B38 (GND), J3.B39 (GND), J3.B6 (GND), J3.B7 (GND), J3.C1 (GND), J3.C12 (GND), J3.C13 (GND), J3.C16 (GND), J3.C17 (GND), J3.C20 (GND), J3.C21 (GND), J3.C24 (GND), J3.C25 (GND), J3.C28 (GND), J3.C29 (GND), J3.C32 (GND), J3.C33 (GND), J3.C36 (GND), J3.C38 (GND), J3.C4 (GND), J3.C40 (GND), J3.C5 (GND), J3.C8 (GND), J3.C9 (GND), J3.D10 (GND), J3.D13 (GND), J3.D16 (GND), J3.D19 (GND), J3.D2 (GND), J3.D22 (GND), J3.D25 (GND), J3.D28 (GND), J3.D3 (GND), J3.D37 (GND), J3.D39 (GND), J3.D6 (GND), J3.D7 (GND), J3.E1 (GND), J3.E11 (GND), J3.E14 (GND), J3.E17 (GND), J3.E20 (GND), J3.E23 (GND), J3.E26 (GND), J3.E29 (GND), J3.E32 (GND), J3.E35 (GND), J3.E38 (GND), J3.E4 (GND), J3.E40 (GND), J3.E5 (GND), J3.E8 (GND), J3.F12 (GND), J3.F15 (GND), J3.F18 (GND), J3.F2 (GND), J3.F21 (GND), J3.F24 (GND), J3.F27 (GND), J3.F3 (GND), J3.F30 (GND), J3.F33 (GND), J3.F36 (GND), J3.F39 (GND), J3.F6 (GND), J3.F9 (GND), J3.G1 (GND), J3.G11 (GND), J3.G14 (GND), J3.G17 (GND), J3.G20 (GND), J3.G23 (GND), J3.G26 (GND), J3.G29 (GND), J3.G32 (GND), J3.G35 (GND), J3.G38 (GND), J3.G4 (GND), J3.G40 (GND), J3.G5 (GND), J3.G8 (GND), J3.H12 (GND), J3.H15 (GND), J3.H18 (GND), J3.H21 (GND), J3.H24 (GND), J3.H27 (GND), J3.H3 (GND), J3.H30 (GND), J3.H33 (GND), J3.H36 (GND), J3.H39 (GND), J3.H6 (GND), J3.H9 (GND), J3.J1 (GND), J3.J11 (GND), J3.J14 (GND), J3.J17 (GND), J3.J20 (GND), J3.J23 (GND), J3.J26 (GND), J3.J29 (GND), J3.J32 (GND), J3.J35 (GND), J3.J38 (GND), J3.J4 (GND), J3.J40 (GND), J3.J5 (GND), J3.J8 (GND), J3.K12 (GND), J3.K15 (GND), J3.K18 (GND), J3.K2 (GND), J3.K21 (GND), J3.K24 (GND), J3.K27 (GND), J3.K3 (GND), J3.K30 (GND), J3.K33 (GND), J3.K36 (GND), J3.K39 (GND), J3.K6 (GND), J3.K9 (GND), J4.2 (Pin_2), J5.2 (Ext), J7.2 (Ext), J8.2 (Ext), J9.6 (Pin_6), R1.2, R10.2, R2.2, R28.1, R29.2, R3.2, R40.1, R48.1, R5.2, R6.2, R7.2, R72.2, R73.2, R74.2, R75.2, R76.2, R77.2, R8.2, R9.2, SW1.10, SW1.11, SW1.12, SW1.13, SW1.14, SW1.15, SW1.16, SW1.9, TP2.1, TP3.1, TP4.1, TP5.1, TP6.1, U1.11 (GND), U10.2 (VSS), U11.2 (V-), U11.3 (IN+), U12.2 (DVSS), U12.20 (AVSS), U12.21 (AVSS), U12.24 (DVSS), U13.2 (VSS), U13.6 (A0), U14.4 (V-), U15.3 (GND), U16.6 (GND), U16.8 (GND), U17.6 (GND), U17.7 (GND), U19.1 (GND), U2.11 (GND), U3.11 (GND), U4.11 (GND), U5.11 (GND), U6.2 (V-), U6.3 (IN+), U7.2 (DVSS), U7.20 (AVSS), U7.21 (AVSS), U7.24 (DVSS), U8.11 (GND), U9.6 (*EN), U9.7 (VSS), U9.8 (GND)
Changed lines of the file:
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@@
 	)
 	(junction
-		(at 543.56 55.88)
-		(diameter 0)
-		(color 0 0 0 0)
-	)
-	(junction
 		(at 641.35 359.41)
 		(diameter 0)
@@
 	)
 	(junction
-		(at 568.96 63.5)
-		(diameter 0)
-		(color 0 0 0 0)
-	)
-	(junction
 		(at 572.77 349.25)
 		(diameter 0)
@@
 	(wire
 		(pts
-			(xy 543.56 63.5) (xy 568.96 63.5)
-		)
-		(stroke
-			(width 0)
-			(type default)
-		)
-	)
-	(wire
-		(pts
 			(xy 347.98 397.51) (xy 358.14 397.51)
 		)
@@
 	(wire
 		(pts
-			(xy 543.56 55.88) (xy 543.56 63.5)
-		)
-		(stroke
-			(width 0)
-			(type default)
-		)
-	)
-	(wire
-		(pts
 			(xy 38.1 119.38) (xy 38.1 129.54)
 		)
@@
 			)
 		)
-		(property "Footprint" "VSSOP8_DGK_TEX"
+		(property "Footprint" "offramps_lib:VSSOP8_DGK_TEX"
 			(at 541.02 205.74 0)
 			(effects

Commit message: Some routing
Parts:
- removed R50, R51, R55, R56: 10K, Resistor_SMD:R_0805_2012Metric, symbol Device:R
